File: rf_autt.sch (KiCad schematic (older format))
At the start: 0 parts

Commit message: Attenuator revised
Parts:
- added R?: 33, symbol Device:R
- added R? (x2): 27, symbol Device:R
- added R?: 3, symbol Device:R
- added R? (x2): 47, symbol Device:R
- added R?: 10, symbol Device:R
- added R? (x2): 39, symbol Device:R
- added U?: FST3253, symbol sdr:FST3253
Connections:
- new net: R?.1, R?.2, R?.2 (x3)
- new net 0dB: U?.10 (2B1), U?.6 (1B1)
- new net 10dB_in: R?.2, U?.5 (1B2)
- new net 10dB_out: R?.1, U?.11 (2B2)
- new net 20dB_in: R?.2, U?.4 (1B3)
- new net 20dB_out: R?.1, U?.12 (2B3)
- new net 30dB_in: R?.2, U?.3 (1B4)
- new net 30dB_out: R?.1, U?.13 (2B4)
- new net ATT_SEL0: U?.14 (S0)
- new net ATT_SEL1: U?.2 (S1)
- new net GNDA: R?.1, R?.1, R?.1
- new net GNDD: U?.1 (~OE1), U?.15 (~OE2), U?.8 (GND)
- new net IN: U?.7 (1A)
- new net OUT: U?.9 (2A)
- new net VCC: U?.16 (VCC)
Other:
- note added: "0 dB"
- note added: "10 dB"
- note added: "20 dB"
- note added: "30 dB"
- note added: "S0 S1 Att\n\n 0 0 0dB\n 0 1 10dB\n 1 0 20dB\n 1 1 30dB"
