File: if1_bpf.sch (KiCad schematic (older format))
At the start: 0 parts

Commit message: 37.4Mega
Parts:
- added C?: 33p, symbol Device:C
- added C?: 470p, symbol Device:C
- added C?: 15p, symbol Device:C
- added C?: 220p, symbol Device:C
- added L?: 560n, symbol Device:L
- added L?: 39n, symbol Device:L
- added L?: 1.2u, symbol Device:L
- added L?: 82n, symbol Device:L
Connections:
- new net: C?.1, L?.2 (x2)
- new net: C?.2, C?.2, L?.1, L?.1
- new net GND: C?.1, C?.1, L?.2, L?.2
- new net IN: C?.2
- new net OUT: C?.2, L?.1, L?.1
Changed lines of the file:
@@
 $Descr A4 11693 8268
 encoding utf-8
-Sheet 4 7
+Sheet 3 7
 Title ""
 Date ""
@@
 Comment4 ""
 $EndDescr
+$Comp
+L Device:C C?
+U 1 1 5FE7343E
+P 3250 2000
+F 0 "C?" V 2998 2000 50  0000 C CNN
+F 1 "33p" V 3089 2000 50  0000 C CNN
+F 2 "" H 3288 1850 50  0001 C CNN
+F 3 "~" H 3250 2000 50  0001 C CNN
+	1    3250 2000
+	0    1    1    0
+$EndComp
+$Comp
+L Device:L L?
+U 1 1 5FE73D0E
+P 3650 2000
+F 0 "L?" V 3840 2000 50  0000 C CNN
+F 1 "560n" V 3749 2000 50  0000 C CNN
+F 2 "" H 3650 2000 50  0001 C CNN
+F 3 "~" H 3650 2000 50  0001 C CNN
+	1    3650 2000
+	0    1    -1   0
+$EndComp
+$Comp
+L Device:C C?
+U 1 1 5FE74A56
+P 3900 2150
+F 0 "C?" H 3785 2104 50  0000 R CNN
+F 1 "470p" H 3785 2195 50  0000 R CNN
+F 2 "" H 3938 2000 50  0001 C CNN
+F 3 "~" H 3900 2150 50  0001 C CNN
+	1    3900 2150
+	-1   0    0    1
+$EndComp
+$Comp
+L Device:L L?
+U 1 1 5FE75044
+P 4300 2150
+F 0 "L?" H 4352 2196 50  0000 L CNN
+F 1 "39n" H 4352 2105 50  0000 L CNN
+F 2 "" H 4300 2150 50  0001 C CNN
+F 3 "~" H 4300 2150 50  0001 C CNN
+	1    4300 2150
+	1    0    0    -1
+$EndComp
+$Comp
+L Device:C C?
+U 1 1 5FE756D3
+P 4650 2000
+F 0 "C?" V 4398 2000 50  0000 C CNN
+F 1 "15p" V 4489 2000 50  0000 C CNN
+F 2 "" H 4688 1850 50  0001 C CNN
+F 3 "~" H 4650 2000 50  0001 C CNN
+	1    4650 2000
+	0    1    1    0
+$EndComp
+$Comp
+L Device:L L?
+U 1 1 5FE771FA
+P 5050 2000
+F 0 "L?" V 5240 2000 50  0000 C CNN
+F 1 "1.2u" V 5149 2000 50  0000 C CNN
+F 2 "" H 5050 2000 50  0001 C CNN
+F 3 "~" H 5050 2000 50  0001 C CNN
+	1    5050 2000
+	0    1    -1   0
+$EndComp
+$Comp
+L Device:L L?
+U 1 1 5FE79301
+P 5700 2150
+F 0 "L?" H 5752 2196 50  0000 L CNN
+F 1 "82n" H 5752 2105 50  0000 L CNN
+F 2 "" H 5700 2150 50  0001 C CNN
+F 3 "~" H 5700 2150 50  0001 C CNN
+	1    5700 2150
+	1    0    0    -1
+$EndComp
+$Comp
+L Device:C C?
+U 1 1 5FE792FB
+P 5300 2150
+F 0 "C?" H 5185 2104 50  0000 R CNN
+F 1 "220p" H 5185 2195 50  0000 R CNN
+F 2 "" H 5338 2000 50  0001 C CNN
+F 3 "~" H 5300 2150 50  0001 C CNN
+	1    5300 2150
+	-1   0    0    1
+$EndComp
+Wire Wire Line
+	2950 2000 3100 2000
+Wire Wire Line
+	3400 2000 3500 2000
+Wire Wire Line
+	3800 2000 3900 2000
+Connection ~ 3900 2000
+Wire Wire Line
+	3900 2000 4300 2000
+Connection ~ 4300 2000
+Wire Wire Line
+	4300 2000 4500 2000
+Wire Wire Line
+	4800 2000 4900 2000
+Wire Wire Line
+	5200 2000 5300 2000
+Connection ~ 5300 2000
+Wire Wire Line
+	5300 2000 5700 2000
+$Comp
+L power:GND #PWR?
+U 1 1 5FE7C471
+P 3900 2300
+F 0 "#PWR?" H 3900 2050 50  0001 C CNN
+F 1 "GND" H 3905 2127 50  0000 C CNN
+F 2 "" H 3900 2300 50  0001 C CNN
+F 3 "" H 3900 2300 50  0001 C CNN
+	1    3900 2300
+	1    0    0    -1
+$EndComp
+$Comp
+L power:GND #PWR?
+U 1 1 5FE7C8C8
+P 4300 2300
+F 0 "#PWR?" H 4300 2050 50  0001 C CNN
+F 1 "GND" H 4305 2127 50  0000 C CNN
+F 2 "" H 4300 2300 50  0001 C CNN
+F 3 "" H 4300 2300 50  0001 C CNN
+	1    4300 2300
+	1    0    0    -1
+$EndComp
+$Comp
+L power:GND #PWR?
+U 1 1 5FE7CE31
+P 5300 2300
+F 0 "#PWR?" H 5300 2050 50  0001 C CNN
+F 1 "GND" H 5305 2127 50  0000 C CNN
+F 2 "" H 5300 2300 50  0001 C CNN
+F 3 "" H 5300 2300 50  0001 C CNN
+	1    5300 2300
+	1    0    0    -1
+$EndComp
+$Comp
+L power:GND #PWR?
+U 1 1 5FE7D2D1
+P 5700 2300
+F 0 "#PWR?" H 5700 2050 50  0001 C CNN
+F 1 "GND" H 5705 2127 50  0000 C CNN
+F 2 "" H 5700 2300 50  0001 C CNN
+F 3 "" H 5700 2300 50  0001 C CNN
+	1    5700 2300
+	1    0    0    -1
+$EndComp
+Text HLabel 2950 2000 0    50   Input ~ 0
+IN
+Text HLabel 5700 2000 2    50   Input ~ 0
+OUT
 $EndSCHEMATC
