File: if2_amp.sch (KiCad schematic (older format))
At the start: 14 parts

Commit message: Initalize receiver test circuit
Parts:
- gave numbers to parts that had none: 14
Connections:
- wire segments 45 -> 46
Changed lines of the file:
@@
 $Descr A4 11693 8268
 encoding utf-8
-Sheet 6 9
+Sheet 6 7
 Title ""
 Date ""
@@
 $EndDescr
 $Comp
-L sdr:MCP6D11 U?
+L sdr:MCP6D11 U3
 U 1 1 5FEA4D4E
 P 2450 3150
-F 0 "U?" H 2400 4250 50  0000 C CNN
+F 0 "U3" H 2400 4250 50  0000 C CNN
 F 1 "MCP6D11" H 2400 4150 50  0000 C CNN
 F 2 "Package_SO:MSOP-8_3x3mm_P0.65mm" H 2400 3000 50  0001 L CNN
@@
 	2500 2850 2400 2850
 $Comp
-L power:GND #PWR?
+L power:GND #PWR0128
 U 1 1 5FEAC1C0
 P 2400 3450
-F 0 "#PWR?" H 2400 3200 50  0001 C CNN
+F 0 "#PWR0128" H 2400 3200 50  0001 C CNN
 F 1 "GND" H 2400 3300 50  0000 C CNN
 F 2 "" H 2400 3450 50  0001 C CNN
@@
 $EndComp
 $Comp
-L Device:R R?
+L Device:R R9
 U 1 1 5FEAD645
 P 2400 2450
-F 0 "R?" V 2193 2450 50  0000 C CNN
+F 0 "R9" V 2193 2450 50  0000 C CNN
 F 1 "10k" V 2284 2450 50  0000 C CNN
 F 2 "" V 2330 2450 50  0001 C CNN
@@
 $EndComp
 $Comp
-L Device:R R?
+L Device:R R10
 U 1 1 5FEAE12B
 P 2400 3850
-F 0 "R?" V 2600 3850 50  0000 C CNN
+F 0 "R10" V 2600 3850 50  0000 C CNN
 F 1 "10k" V 2500 3850 50  0000 C CNN
 F 2 "" V 2330 3850 50  0001 C CNN
@@
 	2800 3150 2750 3150
 $Comp
-L power:+5VA #PWR?
+L power:+5VA #PWR0129
 U 1 1 5FEB0DF4
 P 2400 2850
-F 0 "#PWR?" H 2400 2700 50  0001 C CNN
+F 0 "#PWR0129" H 2400 2700 50  0001 C CNN
 F 1 "+5VA" H 2415 3023 50  0000 C CNN
 F 2 "" H 2400 2850 50  0001 C CNN
@@
 Connection ~ 2400 2850
 $Comp
-L power:+5VA #PWR?
+L power:+5VA #PWR0130
 U 1 1 5FEB1889
 P 4000 2200
-F 0 "#PWR?" H 4000 2050 50  0001 C CNN
+F 0 "#PWR0130" H 4000 2050 50  0001 C CNN
 F 1 "+5VA" H 4015 2373 50  0000 C CNN
 F 2 "" H 4000 2200 50  0001 C CNN
@@
 $EndComp
 $Comp
-L Device:R R?
+L Device:R R11
 U 1 1 5FEB1EAA
 P 4000 2350
-F 0 "R?" H 4070 2396 50  0000 L CNN
+F 0 "R11" H 4070 2396 50  0000 L CNN
 F 1 "100k" H 4070 2305 50  0000 L CNN
 F 2 "" V 3930 2350 50  0001 C CNN
@@
 $EndComp
 $Comp
-L Device:R R?
+L Device:R R12
 U 1 1 5FEB22B7
 P 4000 2750
-F 0 "R?" H 4070 2796 50  0000 L CNN
+F 0 "R12" H 4070 2796 50  0000 L CNN
 F 1 "100k" H 4070 2705 50  0000 L CNN
 F 2 "" V 3930 2750 50  0001 C CNN
@@
 $EndComp
 $Comp
-L power:GND #PWR?
+L power:GND #PWR0131
 U 1 1 5FEB26F6
 P 4000 2900
-F 0 "#PWR?" H 4000 2650 50  0001 C CNN
+F 0 "#PWR0131" H 4000 2650 50  0001 C CNN
 F 1 "GND" H 4000 2750 50  0000 C CNN
 F 2 "" H 4000 2900 50  0001 C CNN
@@
 The previous filter has 750 ohm output impedance\n
 $Comp
-L Device:Q_NPN_BCE Q?
+L Device:Q_NPN_BCE Q2
 U 1 1 5FEBCF7E
 P 6800 4650
-F 0 "Q?" H 6991 4696 50  0000 L CNN
+F 0 "Q2" H 6991 4696 50  0000 L CNN
 F 1 "Q_NPN_BCE" H 6991 4605 50  0000 L CNN
 F 2 "" H 7000 4750 50  0001 C CNN
@@
 $EndComp
 $Comp
-L Device:Q_NPN_BCE Q?
+L Device:Q_NPN_BCE Q3
 U 1 1 5FEBD9DD
 P 7650 4650
-F 0 "Q?" H 7841 4696 50  0000 L CNN
+F 0 "Q3" H 7841 4696 50  0000 L CNN
 F 1 "Q_NPN_BCE" H 7841 4605 50  0000 L CNN
 F 2 "" H 7850 4750 50  0001 C CNN
@@
 $EndComp
 $Comp
-L Device:C C?
+L Device:C C32
 U 1 1 5FEBE468
 P 7250 5050
-F 0 "C?" H 7365 5096 50  0000 L CNN
+F 0 "C32" H 7365 5096 50  0000 L CNN
 F 1 "C" H 7365 5005 50  0000 L CNN
 F 2 "" H 7288 4900 50  0001 C CNN
@@
 $EndComp
 $Comp
-L power:GNDA #PWR?
+L power:GNDA #PWR0132
 U 1 1 5FEBEF6E
 P 7250 5200
-F 0 "#PWR?" H 7250 4950 50  0001 C CNN
+F 0 "#PWR0132" H 7250 4950 50  0001 C CNN
 F 1 "GNDA" H 7255 5027 50  0000 C CNN
 F 2 "" H 7250 5200 50  0001 C CNN
@@
 	7250 4650 7400 4650
 $Comp
-L Device:R R?
+L Device:R R14
 U 1 1 5FEBFA1D
 P 8850 4200
-F 0 "R?" H 8920 4246 50  0000 L CNN
+F 0 "R14" H 8920 4246 50  0000 L CNN
 F 1 "R" H 8920 4155 50  0000 L CNN
 F 2 "" V 8780 4200 50  0001 C CNN
@@
 $EndComp
 $Comp
-L Device:R R?
+L Device:R R15
 U 1 1 5FEBFCA7
 P 8850 4500
-F 0 "R?" H 8920 4546 50  0000 L CNN
+F 0 "R15" H 8920 4546 50  0000 L CNN
 F 1 "R" H 8920 4455 50  0000 L CNN
 F 2 "" V 8780 4500 50  0001 C CNN
@@
 $EndComp
 $Comp
-L power:GNDA #PWR?
+L power:GNDA #PWR0133
 U 1 1 5FEC0155
 P 8850 4650
-F 0 "#PWR?" H 8850 4400 50  0001 C CNN
+F 0 "#PWR0133" H 8850 4400 50  0001 C CNN
 F 1 "GNDA" H 8855 4477 50  0000 C CNN
 F 2 "" H 8850 4650 50  0001 C CNN
@@
 	6700 4850 6700 5200
 $Comp
-L Device:R R?
+L Device:R R13
 U 1 1 5FEC59DE
 P 6850 5900
-F 0 "R?" V 6643 5900 50  0000 C CNN
+F 0 "R13" V 6643 5900 50  0000 C CNN
 F 1 "R" V 6734 5900 50  0000 C CNN
 F 2 "" V 6780 5900 50  0001 C CNN
@@
 $EndComp
 $Comp
-L power:GNDA #PWR?
+L power:GNDA #PWR0134
 U 1 1 5FEC63DD
 P 7000 5900
-F 0 "#PWR?" H 7000 5650 50  0001 C CNN
+F 0 "#PWR0134" H 7000 5650 50  0001 C CNN
 F 1 "GNDA" H 7005 5727 50  0000 C CNN
 F 2 "" H 7000 5900 50  0001 C CNN
@@
 $EndComp
 $Comp
-L Device:L L?
+L Device:L L18
 U 1 1 5FEC71FC
 P 6700 3650
-F 0 "L?" H 6753 3696 50  0000 L CNN
+F 0 "L18" H 6753 3696 50  0000 L CNN
 F 1 "L" H 6753 3605 50  0000 L CNN
 F 2 "" H 6700 3650 50  0001 C CNN
@@
 $EndComp
 $Comp
-L Device:C C?
+L Device:C C31
 U 1 1 5FEC7CF1
 P 7200 4200
-F 0 "C?" H 7315 4246 50  0000 L CNN
+F 0 "C31" H 7315 4246 50  0000 L CNN
 F 1 "C" H 7315 4155 50  0000 L CNN
 F 2 "" H 7238 4050 50  0001 C CNN
@@
 $EndComp
 $Comp
-L Device:L L?
+L Device:L L19
 U 1 1 5FEC838F
 P 7750 3650
-F 0 "L?" H 7803 3696 50  0000 L CNN
+F 0 "L19" H 7803 3696 50  0000 L CNN
 F 1 "L" H 7803 3605 50  0000 L CNN
 F 2 "" H 7750 3650 50  0001 C CNN
@@
 	8850 4050 8850 3200
 Wire Wire Line
-	8850 3200 7250 3200
+	8850 3200 8100 3200
 Wire Wire Line
 	7250 3200 7250 3500
@@
 Text HLabel 6700 5900 0    50   Input ~ 0
 DC_CM
+$Comp
+L power:+5VA #PWR0135
+U 1 1 5FFA269D
+P 8100 3200
+F 0 "#PWR0135" H 8100 3050 50  0001 C CNN
+F 1 "+5VA" H 8115 3373 50  0000 C CNN
+F 2 "" H 8100 3200 50  0001 C CNN
+F 3 "" H 8100 3200 50  0001 C CNN
+	1    8100 3200
+	1    0    0    -1
+$EndComp
+Connection ~ 8100 3200
+Wire Wire Line
+	8100 3200 7250 3200
 $EndSCHEMATC

Commit message: Nyáktervezésre majdnem kész
Parts:
- removed R11: 100k, symbol Device:R
- added R35, R36, R37, R38, R39: BP, Resistor_SMD:R_1206_3216Metric_Pad1.42x1.75mm_HandSolder, symbol Device:R
- C31, C32: footprint (none) -> Capacitor_SMD:C_0805_2012Metric_Pad1.15x1.40mm_HandSolder
- R10, R9: value 10k -> 1.2k; footprint (none) -> Resistor_SMD:R_0805_2012Metric_Pad1.15x1.40mm_HandSolder
- R12: value 100k -> BP; footprint (none) -> Resistor_SMD:R_1206_3216Metric_Pad1.42x1.75mm_HandSolder
- R13, R14, R15: footprint (none) -> Resistor_SMD:R_0805_2012Metric_Pad1.15x1.40mm_HandSolder
Connections:
- net labels removed: 2.5V
- wire segments 46 -> 44
Other:
- note removed: "If we want to compensate for the previous filter's attenuation, we need a 26k resistor in order to have in total 30.8 dB gain\n"
- note removed: "The previous filter has 750 ohm output impedance\n"
- note removed: "This way, we have exactly 22dB\n"
Changed lines of the file:
@@
 	1    0    0    -1
 $EndComp
-Text HLabel 6700 5200 0    50   Input ~ 0
+Text HLabel 6100 5200 0    50   Input ~ 0
 In+
-Text HLabel 6700 5500 0    50   Input ~ 0
+Text HLabel 6100 5500 0    50   Input ~ 0
 In-
 Wire Wire Line
@@
 P 2400 2450
 F 0 "R9" V 2193 2450 50  0000 C CNN
-F 1 "10k" V 2284 2450 50  0000 C CNN
-F 2 "" V 2330 2450 50  0001 C CNN
+F 1 "1.2k" V 2284 2450 50  0000 C CNN
+F 2 "Resistor_SMD:R_0805_2012Metric_Pad1.15x1.40mm_HandSolder" V 2330 2450 50  0001 C CNN
 F 3 "~" H 2400 2450 50  0001 C CNN
 	1    2400 2450
@@
 P 2400 3850
 F 0 "R10" V 2600 3850 50  0000 C CNN
-F 1 "10k" V 2500 3850 50  0000 C CNN
-F 2 "" V 2330 3850 50  0001 C CNN
+F 1 "1.2k" V 2500 3850 50  0000 C CNN
+F 2 "Resistor_SMD:R_0805_2012Metric_Pad1.15x1.40mm_HandSolder" V 2330 3850 50  0001 C CNN
 F 3 "~" H 2400 3850 50  0001 C CNN
 	1    2400 3850
@@
 $EndComp
 Connection ~ 2400 2850
-$Comp
-L power:+5VA #PWR0130
-U 1 1 5FEB1889
-P 4000 2200
-F 0 "#PWR0130" H 4000 2050 50  0001 C CNN
-F 1 "+5VA" H 4015 2373 50  0000 C CNN
-F 2 "" H 4000 2200 50  0001 C CNN
-F 3 "" H 4000 2200 50  0001 C CNN
-	1    4000 2200
-	1    0    0    -1
-$EndComp
-$Comp
-L Device:R R11
-U 1 1 5FEB1EAA
-P 4000 2350
-F 0 "R11" H 4070 2396 50  0000 L CNN
-F 1 "100k" H 4070 2305 50  0000 L CNN
-F 2 "" V 3930 2350 50  0001 C CNN
-F 3 "~" H 4000 2350 50  0001 C CNN
-	1    4000 2350
-	1    0    0    -1
-$EndComp
-$Comp
-L Device:R R12
-U 1 1 5FEB22B7
-P 4000 2750
-F 0 "R12" H 4070 2796 50  0000 L CNN
-F 1 "100k" H 4070 2705 50  0000 L CNN
-F 2 "" V 3930 2750 50  0001 C CNN
-F 3 "~" H 4000 2750 50  0001 C CNN
-	1    4000 2750
-	1    0    0    -1
-$EndComp
-$Comp
-L power:GND #PWR0131
-U 1 1 5FEB26F6
-P 4000 2900
-F 0 "#PWR0131" H 4000 2650 50  0001 C CNN
-F 1 "GND" H 4000 2750 50  0000 C CNN
-F 2 "" H 4000 2900 50  0001 C CNN
-F 3 "" H 4000 2900 50  0001 C CNN
-	1    4000 2900
-	1    0    0    -1
-$EndComp
-Text GLabel 2800 3150 2    50   Input ~ 0
-2.5V
-Text GLabel 4050 2550 2    50   Input ~ 0
-2.5V
-Wire Wire Line
-	4000 2500 4000 2550
-Wire Wire Line
-	4000 2550 4050 2550
-Connection ~ 4000 2550
-Wire Wire Line
-	4000 2550 4000 2600
-Text Notes 1250 1350 0    50   ~ 0
-If we want to compensate for the previous filter's attenuation, we need a 26k resistor in order to have in total 30.8 dB gain\n
-Text Notes 1250 1500 0    50   ~ 0
-This way, we have exactly 22dB\n
-Text Notes 1250 1650 0    50   ~ 0
-The previous filter has 750 ohm output impedance\n
 $Comp
 L Device:Q_NPN_BCE Q2
@@
 F 0 "C32" H 7365 5096 50  0000 L CNN
 F 1 "C" H 7365 5005 50  0000 L CNN
-F 2 "" H 7288 4900 50  0001 C CNN
+F 2 "Capacitor_SMD:C_0805_2012Metric_Pad1.15x1.40mm_HandSolder" H 7288 4900 50  0001 C CNN
 F 3 "~" H 7250 5050 50  0001 C CNN
 	1    7250 5050
@@
 F 0 "R14" H 8920 4246 50  0000 L CNN
 F 1 "R" H 8920 4155 50  0000 L CNN
-F 2 "" V 8780 4200 50  0001 C CNN
+F 2 "Resistor_SMD:R_0805_2012Metric_Pad1.15x1.40mm_HandSolder" V 8780 4200 50  0001 C CNN
 F 3 "~" H 8850 4200 50  0001 C CNN
 	1    8850 4200
@@
 F 0 "R15" H 8920 4546 50  0000 L CNN
 F 1 "R" H 8920 4455 50  0000 L CNN
-F 2 "" V 8780 4500 50  0001 C CNN
+F 2 "Resistor_SMD:R_0805_2012Metric_Pad1.15x1.40mm_HandSolder" V 8780 4500 50  0001 C CNN
 F 3 "~" H 8850 4500 50  0001 C CNN
 	1    8850 4500
@@
 	6700 4850 6700 5200
 $Comp
-L Device:R R13
-U 1 1 5FEC59DE
-P 6850 5900
-F 0 "R13" V 6643 5900 50  0000 C CNN
-F 1 "R" V 6734 5900 50  0000 C CNN
-F 2 "" V 6780 5900 50  0001 C CNN
-F 3 "~" H 6850 5900 50  0001 C CNN
-	1    6850 5900
-	0    1    1    0
-$EndComp
+L Device:L L18
+U 1 1 5FEC71FC
+P 6700 3650
+F 0 "L18" H 6753 3696 50  0000 L CNN
+F 1 "L" H 6753 3605 50  0000 L CNN
+F 2 "" H 6700 3650 50  0001 C CNN
+F 3 "~" H 6700 3650 50  0001 C CNN
+	1    6700 3650
+	1    0    0    -1
+$EndComp
+$Comp
+L Device:C C31
+U 1 1 5FEC7CF1
+P 7200 4200
+F 0 "C31" H 7315 4246 50  0000 L CNN
+F 1 "C" H 7315 4155 50  0000 L CNN
+F 2 "Capacitor_SMD:C_0805_2012Metric_Pad1.15x1.40mm_HandSolder" H 7238 4050 50  0001 C CNN
+F 3 "~" H 7200 4200 50  0001 C CNN
+	1    7200 4200
+	0    1    1    0
+$EndComp
+$Comp
+L Device:L L19
+U 1 1 5FEC838F
+P 7750 3650
+F 0 "L19" H 7803 3696 50  0000 L CNN
+F 1 "L" H 7803 3605 50  0000 L CNN
+F 2 "" H 7750 3650 50  0001 C CNN
+F 3 "~" H 7750 3650 50  0001 C CNN
+	1    7750 3650
+	1    0    0    -1
+$EndComp
+Wire Wire Line
+	6700 3500 7250 3500
+Wire Wire Line
+	8850 4050 8850 3200
+Wire Wire Line
+	8850 3200 8100 3200
+Wire Wire Line
+	7250 3200 7250 3500
+Connection ~ 7250 3500
+Wire Wire Line
+	7250 3500 7750 3500
+Wire Wire Line
+	7750 3950 10350 3950
+Connection ~ 7750 3950
+Wire Wire Line
+	7750 3950 7750 3800
+Wire Wire Line
+	6700 3850 10350 3850
+Connection ~ 6700 3850
+Wire Wire Line
+	6700 3850 6700 3800
+Wire Wire Line
+	6700 3850 6700 4200
+Wire Wire Line
+	7350 4200 7750 4200
+Wire Wire Line
+	7750 3950 7750 4200
+Connection ~ 7750 4200
+Wire Wire Line
+	7750 4200 7750 4450
+Wire Wire Line
+	7050 4200 6700 4200
+Connection ~ 6700 4200
+Wire Wire Line
+	6700 4200 6700 4450
+Wire Wire Line
+	7750 5500 7750 4850
+$Comp
+L power:+5VA #PWR0135
+U 1 1 5FFA269D
+P 8100 3200
+F 0 "#PWR0135" H 8100 3050 50  0001 C CNN
+F 1 "+5VA" H 8115 3373 50  0000 C CNN
+F 2 "" H 8100 3200 50  0001 C CNN
+F 3 "" H 8100 3200 50  0001 C CNN
+	1    8100 3200
+	1    0    0    -1
+$EndComp
+Connection ~ 8100 3200
+Wire Wire Line
+	8100 3200 7250 3200
+Text HLabel 6700 5900 0    50   Input ~ 0
+DC_CM
 $Comp
 L power:GNDA #PWR0134
@@
 $EndComp
 $Comp
-L Device:L L18
-U 1 1 5FEC71FC
-P 6700 3650
-F 0 "L18" H 6753 3696 50  0000 L CNN
-F 1 "L" H 6753 3605 50  0000 L CNN
-F 2 "" H 6700 3650 50  0001 C CNN
-F 3 "~" H 6700 3650 50  0001 C CNN
-	1    6700 3650
-	1    0    0    -1
-$EndComp
-$Comp
-L Device:C C31
-U 1 1 5FEC7CF1
-P 7200 4200
-F 0 "C31" H 7315 4246 50  0000 L CNN
-F 1 "C" H 7315 4155 50  0000 L CNN
-F 2 "" H 7238 4050 50  0001 C CNN
-F 3 "~" H 7200 4200 50  0001 C CNN
-	1    7200 4200
-	0    1    1    0
-$EndComp
-$Comp
-L Device:L L19
-U 1 1 5FEC838F
-P 7750 3650
-F 0 "L19" H 7803 3696 50  0000 L CNN
-F 1 "L" H 7803 3605 50  0000 L CNN
-F 2 "" H 7750 3650 50  0001 C CNN
-F 3 "~" H 7750 3650 50  0001 C CNN
-	1    7750 3650
-	1    0    0    -1
-$EndComp
-Wire Wire Line
-	6700 3500 7250 3500
-Wire Wire Line
-	8850 4050 8850 3200
-Wire Wire Line
-	8850 3200 8100 3200
-Wire Wire Line
-	7250 3200 7250 3500
-Connection ~ 7250 3500
-Wire Wire Line
-	7250 3500 7750 3500
-Wire Wire Line
-	7750 3950 10400 3950
-Connection ~ 7750 3950
-Wire Wire Line
-	7750 3950 7750 3800
-Wire Wire Line
-	6700 3850 10350 3850
-Connection ~ 6700 3850
-Wire Wire Line
-	6700 3850 6700 3800
-Wire Wire Line
-	6700 3850 6700 4200
-Wire Wire Line
-	7350 4200 7750 4200
-Wire Wire Line
-	7750 3950 7750 4200
-Connection ~ 7750 4200
-Wire Wire Line
-	7750 4200 7750 4450
-Wire Wire Line
-	7050 4200 6700 4200
-Connection ~ 6700 4200
-Wire Wire Line
-	6700 4200 6700 4450
-Wire Wire Line
-	7750 5500 7750 4850
-Wire Wire Line
-	6700 5500 7750 5500
-Text HLabel 6700 5900 0    50   Input ~ 0
+L Device:R R13
+U 1 1 5FEC59DE
+P 6850 5900
+F 0 "R13" V 6643 5900 50  0000 C CNN
+F 1 "R" V 6734 5900 50  0000 C CNN
+F 2 "Resistor_SMD:R_0805_2012Metric_Pad1.15x1.40mm_HandSolder" V 6780 5900 50  0001 C CNN
+F 3 "~" H 6850 5900 50  0001 C CNN
+	1    6850 5900
+	0    1    1    0
+$EndComp
+Text HLabel 2800 3150 2    50   Input ~ 0
 DC_CM
-$Comp
-L power:+5VA #PWR0135
-U 1 1 5FFA269D
-P 8100 3200
-F 0 "#PWR0135" H 8100 3050 50  0001 C CNN
-F 1 "+5VA" H 8115 3373 50  0000 C CNN
-F 2 "" H 8100 3200 50  0001 C CNN
-F 3 "" H 8100 3200 50  0001 C CNN
-	1    8100 3200
-	1    0    0    -1
-$EndComp
-Connection ~ 8100 3200
-Wire Wire Line
-	8100 3200 7250 3200
+Text HLabel 1500 3250 0    50   Input ~ 0
+In+
+Text HLabel 1500 3050 0    50   Input ~ 0
+In-
+$Comp
+L Device:R R12
+U 1 1 5FFCBAF5
+P 1650 3050
+F 0 "R12" V 1443 3050 50  0000 C CNN
+F 1 "BP" V 1534 3050 50  0000 C CNN
+F 2 "Resistor_SMD:R_1206_3216Metric_Pad1.42x1.75mm_HandSolder" V 1580 3050 50  0001 C CNN
+F 3 "~" H 1650 3050 50  0001 C CNN
+	1    1650 3050
+	0    1    1    0
+$EndComp
+$Comp
+L Device:R R35
+U 1 1 5FFCD24E
+P 1650 3250
+F 0 "R35" V 1443 3250 50  0000 C CNN
+F 1 "BP" V 1534 3250 50  0000 C CNN
+F 2 "Resistor_SMD:R_1206_3216Metric_Pad1.42x1.75mm_HandSolder" V 1580 3250 50  0001 C CNN
+F 3 "~" H 1650 3250 50  0001 C CNN
+	1    1650 3250
+	0    1    1    0
+$EndComp
+$Comp
+L Device:R R36
+U 1 1 5FFCD441
+P 6250 5200
+F 0 "R36" V 6043 5200 50  0000 C CNN
+F 1 "BP" V 6134 5200 50  0000 C CNN
+F 2 "Resistor_SMD:R_1206_3216Metric_Pad1.42x1.75mm_HandSolder" V 6180 5200 50  0001 C CNN
+F 3 "~" H 6250 5200 50  0001 C CNN
+	1    6250 5200
+	0    1    1    0
+$EndComp
+Wire Wire Line
+	6400 5200 6700 5200
+$Comp
+L Device:R R37
+U 1 1 5FFCFA23
+P 6250 5500
+F 0 "R37" V 6043 5500 50  0000 C CNN
+F 1 "BP" V 6134 5500 50  0000 C CNN
+F 2 "Resistor_SMD:R_1206_3216Metric_Pad1.42x1.75mm_HandSolder" V 6180 5500 50  0001 C CNN
+F 3 "~" H 6250 5500 50  0001 C CNN
+	1    6250 5500
+	0    1    1    0
+$EndComp
+Wire Wire Line
+	6400 5500 7750 5500
+Text HLabel 10650 3850 2    50   Input ~ 0
+Out+
+Text HLabel 10650 3950 2    50   Input ~ 0
+Out-
+$Comp
+L Device:R R38
+U 1 1 5FFD217D
+P 10500 3850
+F 0 "R38" H 10570 3896 50  0000 L CNN
+F 1 "BP" H 10570 3805 50  0000 L CNN
+F 2 "Resistor_SMD:R_1206_3216Metric_Pad1.42x1.75mm_HandSolder" V 10430 3850 50  0001 C CNN
+F 3 "~" H 10500 3850 50  0001 C CNN
+	1    10500 3850
+	0    1    1    0
+$EndComp
+$Comp
+L Device:R R39
+U 1 1 5FFD2490
+P 10500 3950
+F 0 "R39" H 10570 3996 50  0000 L CNN
+F 1 "BP" H 10570 3905 50  0000 L CNN
+F 2 "Resistor_SMD:R_1206_3216Metric_Pad1.42x1.75mm_HandSolder" V 10430 3950 50  0001 C CNN
+F 3 "~" H 10500 3950 50  0001 C CNN
+	1    10500 3950
+	0    1    1    0
+$EndComp
 $EndSCHEMATC
