File: if2_amp.sch (KiCad schematic (older format))
At the start: 25 parts, among them Q2 BC847BS, U3 MCP6D11

Commit message: FPGA change and new project file
Parts:
- renumbered C32 to C?, C31 to C?, C9 to C?, L18 to L?, L19 to L?, Q2 to Q?, R9 to R?, R10 to R?, R14 to R?, R15 to R?, R13 to R?, R12 to R?, R35 to R?, R36 to R?, R37 to R?, R38 to R?, R39 to R?, R40 to R?, R41 to R?, R42 to R?, U3 to U?

Commit message: PCB is Done... Needs DRC check
Parts:
- removed R?: BP, Resistor_SMD:R_0805_2012Metric_Pad1.20x1.40mm_HandSolder, symbol Device:R
- added R9: BP, Resistor_SMD:R_1206_3216Metric_Pad1.42x1.75mm_HandSolder, symbol Device:R
- gave numbers to parts that had none: 20
Connections:
- net GND is gone; now on net GNDA: C32.2, U3.6 (V-)
- net In-: now also R9.2
- net at R12.2, U3.8 (+): now also R9.1

Commit message: RX PCB revision: Diff amp + Mixer2
Parts:
- removed R14, R20, R21: BP, Resistor_SMD:R_1206_3216Metric_Pad1.30x1.75mm_HandSolder, symbol Device:R
- added C35, C36: 10p, Capacitor_SMD:C_0805_2012Metric_Pad1.15x1.40mm_HandSolder, symbol Device:C
- added R18: 10k, Resistor_SMD:R_0805_2012Metric_Pad1.15x1.40mm_HandSolder, symbol Device:R
- added R26: BP, Resistor_SMD:R_1206_3216Metric_Pad1.42x1.75mm_HandSolder, symbol Device:R
- added TP12, TP13: TestPoint_2Pole, Connector_PinHeader_2.54mm:PinHeader_1x02_P2.54mm_Vertical, symbol Connector:TestPoint_2Pole
- C34: renamed from C40; footprint Capacitor_SMD:C_0805_2012Metric_Pad1.18x1.45mm_HandSolder -> Capacitor_SMD:C_0805_2012Metric_Pad1.15x1.40mm_HandSolder
- C37: renamed from C39; footprint Capacitor_SMD:C_0805_2012Metric_Pad1.18x1.45mm_HandSolder -> Capacitor_SMD:C_0805_2012Metric_Pad1.15x1.40mm_HandSolder
- C38: renamed from C36; footprint Capacitor_SMD:C_0805_2012Metric_Pad1.18x1.45mm_HandSolder -> Capacitor_SMD:C_0805_2012Metric_Pad1.15x1.40mm_HandSolder
- C39: renamed from C37; footprint Capacitor_SMD:C_0805_2012Metric_Pad1.18x1.45mm_HandSolder -> Capacitor_SMD:C_0805_2012Metric_Pad1.15x1.40mm_HandSolder
- C40: renamed from C38; footprint Capacitor_SMD:C_0805_2012Metric_Pad1.18x1.45mm_HandSolder -> Capacitor_SMD:C_0805_2012Metric_Pad1.15x1.40mm_HandSolder
- C41: renamed from C32; footprint Capacitor_SMD:C_0805_2012Metric_Pad1.18x1.45mm_HandSolder -> Capacitor_SMD:C_0805_2012Metric_Pad1.15x1.40mm_HandSolder
- R15: value BP -> 10k; footprint Resistor_SMD:R_1206_3216Metric_Pad1.30x1.75mm_HandSolder -> Resistor_SMD:R_0805_2012Metric_Pad1.15x1.40mm_HandSolder
- R16: renamed from R12; footprint Resistor_SMD:R_0805_2012Metric_Pad1.20x1.40mm_HandSolder -> Resistor_SMD:R_0805_2012Metric_Pad1.15x1.40mm_HandSolder
- R19: renamed from R10; footprint Resistor_SMD:R_1206_3216Metric_Pad1.30x1.75mm_HandSolder -> Resistor_SMD:R_1206_3216Metric_Pad1.42x1.75mm_HandSolder
- R20: renamed from R22; footprint Resistor_SMD:R_0805_2012Metric_Pad1.20x1.40mm_HandSolder -> Resistor_SMD:R_0805_2012Metric_Pad1.15x1.40mm_HandSolder
- R21: renamed from R25; footprint Resistor_SMD:R_0805_2012Metric_Pad1.20x1.40mm_HandSolder -> Resistor_SMD:R_0805_2012Metric_Pad1.15x1.40mm_HandSolder
- R22: renamed from R23; footprint Resistor_SMD:R_0805_2012Metric_Pad1.20x1.40mm_HandSolder -> Resistor_SMD:R_0805_2012Metric_Pad1.15x1.40mm_HandSolder
- R23: renamed from R17; footprint Resistor_SMD:R_1206_3216Metric_Pad1.30x1.75mm_HandSolder -> Resistor_SMD:R_1206_3216Metric_Pad1.42x1.75mm_HandSolder
- R24: renamed from R13; footprint Resistor_SMD:R_0805_2012Metric_Pad1.20x1.40mm_HandSolder -> Resistor_SMD:R_0805_2012Metric_Pad1.15x1.40mm_HandSolder
- R25: renamed from R18; footprint Resistor_SMD:R_1206_3216Metric_Pad1.30x1.75mm_HandSolder -> Resistor_SMD:R_1206_3216Metric_Pad1.42x1.75mm_HandSolder
- R27: renamed from R19; footprint Resistor_SMD:R_0805_2012Metric_Pad1.20x1.40mm_HandSolder -> Resistor_SMD:R_0805_2012Metric_Pad1.15x1.40mm_HandSolder
- R28: renamed from R16; footprint Resistor_SMD:R_0805_2012Metric_Pad1.20x1.40mm_HandSolder -> Resistor_SMD:R_1206_3216Metric_Pad1.42x1.75mm_HandSolder
- renumbered R9 to R17
Connections:
- net Out- is gone; now on an unnamed net: R15.1
- net DC_CM: now also R26.2; no longer R27.2
- net at R16.1, U3.4 (Out+): now also C36.1, R18.1, TP13.1
- net at R24.1, U3.5 (Out-): now also C36.2, R18.2, TP13.2; no longer R15.2
- net at C34.2, L17.1, Q2.6 (C1): now also C35.1, TP12.1
- net at C34.1, L18.2, Q2.3 (C2): now also R15.2, C35.2, TP12.2
- new net: R26.1, R27.2
Other:
- note added: "Szimulált terhelés (ADC)"
- moved on the sheet: C41, R27, R28

Commit message: Nézd meg!
Parts:
- added C42: 10n, Capacitor_SMD:C_0805_2012Metric_Pad1.15x1.40mm_HandSolder, symbol Device:C
- added C43, C44: 100n, Capacitor_SMD:C_0805_2012Metric_Pad1.15x1.40mm_HandSolder, symbol Device:C
- added R38: 100, Resistor_SMD:R_0805_2012Metric_Pad1.15x1.40mm_HandSolder, symbol Device:R
Connections:
- net +5VA: now also C44.1, R38.1; no longer U3.3 (V+), U3.7 (/PD)
- net GNDA: now also C42.2, C43.2, C44.2
- new net Opamp5V: C42.1, C43.1, R38.2, U3.3 (V+), U3.7 (/PD)
Changed lines of the file:
@@
 	2800 2450 2550 2450
-$Comp
-L power:+5VA #PWR032
-U 1 1 5FEB0DF4
-P 2400 2850
-F 0 "#PWR032" H 2400 2700 50  0001 C CNN
-F 1 "+5VA" H 2415 3023 50  0000 C CNN
-F 2 "" H 2400 2850 50  0001 C CNN
-F 3 "" H 2400 2850 50  0001 C CNN
-	1    2400 2850
-	1    0    0    -1
-$EndComp
-Connection ~ 2400 2850
 $Comp
 L Device:C C41
@@
 Wire Wire Line
 	7000 2500 7000 2800
+$Comp
+L Device:C C?
+U 1 1 60165078
+P 3300 1550
+AR Path="/5FE332ED/60165078" Ref="C?"  Part="1"
+AR Path="/5FE3342F/60165078" Ref="C42"  Part="1"
+F 0 "C42" H 3415 1596 50  0000 L CNN
+F 1 "10n" H 3415 1505 50  0000 L CNN
+F 2 "Capacitor_SMD:C_0805_2012Metric_Pad1.15x1.40mm_HandSolder" H 3338 1400 50  0001 C CNN
+F 3 "~" H 3300 1550 50  0001 C CNN
+	1    3300 1550
+	1    0    0    -1
+$EndComp
+$Comp
+L power:GNDA #PWR?
+U 1 1 6016507E
+P 3300 1700
+AR Path="/5FE332ED/6016507E" Ref="#PWR?"  Part="1"
+AR Path="/5FE3342F/6016507E" Ref="#PWR0101"  Part="1"
+F 0 "#PWR0101" H 3300 1450 50  0001 C CNN
+F 1 "GNDA" H 3305 1527 50  0000 C CNN
+F 2 "" H 3300 1700 50  0001 C CNN
+F 3 "" H 3300 1700 50  0001 C CNN
+	1    3300 1700
+	1    0    0    -1
+$EndComp
+Wire Wire Line
+	3150 1400 3300 1400
+$Comp
+L Device:C C?
+U 1 1 60165085
+P 3700 1550
+AR Path="/5FE332ED/60165085" Ref="C?"  Part="1"
+AR Path="/5FE3342F/60165085" Ref="C43"  Part="1"
+F 0 "C43" H 3815 1596 50  0000 L CNN
+F 1 "100n" H 3815 1505 50  0000 L CNN
+F 2 "Capacitor_SMD:C_0805_2012Metric_Pad1.15x1.40mm_HandSolder" H 3738 1400 50  0001 C CNN
+F 3 "~" H 3700 1550 50  0001 C CNN
+	1    3700 1550
+	1    0    0    -1
+$EndComp
+$Comp
+L power:GNDA #PWR?
+U 1 1 6016508B
+P 3700 1700
+AR Path="/5FE332ED/6016508B" Ref="#PWR?"  Part="1"
+AR Path="/5FE3342F/6016508B" Ref="#PWR0102"  Part="1"
+F 0 "#PWR0102" H 3700 1450 50  0001 C CNN
+F 1 "GNDA" H 3705 1527 50  0000 C CNN
+F 2 "" H 3700 1700 50  0001 C CNN
+F 3 "" H 3700 1700 50  0001 C CNN
+	1    3700 1700
+	1    0    0    -1
+$EndComp
+Wire Wire Line
+	3300 1400 3700 1400
+Connection ~ 3300 1400
+$Comp
+L Device:R R?
+U 1 1 60165093
+P 3900 1400
+AR Path="/5FE332ED/60165093" Ref="R?"  Part="1"
+AR Path="/5FE3342F/60165093" Ref="R38"  Part="1"
+F 0 "R38" V 3693 1400 50  0000 C CNN
+F 1 "100" V 3784 1400 50  0000 C CNN
+F 2 "Resistor_SMD:R_0805_2012Metric_Pad1.15x1.40mm_HandSolder" V 3830 1400 50  0001 C CNN
+F 3 "~" H 3900 1400 50  0001 C CNN
+	1    3900 1400
+	0    1    1    0
+$EndComp
+Connection ~ 3700 1400
+$Comp
+L Device:C C?
+U 1 1 6016509A
+P 4150 1550
+AR Path="/5FE332ED/6016509A" Ref="C?"  Part="1"
+AR Path="/5FE3342F/6016509A" Ref="C44"  Part="1"
+F 0 "C44" H 4265 1596 50  0000 L CNN
+F 1 "100n" H 4265 1505 50  0000 L CNN
+F 2 "Capacitor_SMD:C_0805_2012Metric_Pad1.15x1.40mm_HandSolder" H 4188 1400 50  0001 C CNN
+F 3 "~" H 4150 1550 50  0001 C CNN
+	1    4150 1550
+	1    0    0    -1
+$EndComp
+Wire Wire Line
+	4150 1400 4050 1400
+Wire Wire Line
+	4650 1200 4650 1400
+Wire Wire Line
+	4650 1400 4150 1400
+Connection ~ 4150 1400
+Wire Wire Line
+	3750 1400 3700 1400
+$Comp
+L power:+5VA #PWR?
+U 1 1 601650A5
+P 4650 1200
+AR Path="/5FE332ED/601650A5" Ref="#PWR?"  Part="1"
+AR Path="/5FE3342F/601650A5" Ref="#PWR0103"  Part="1"
+F 0 "#PWR0103" H 4650 1050 50  0001 C CNN
+F 1 "+5VA" H 4665 1373 50  0000 C CNN
+F 2 "" H 4650 1200 50  0001 C CNN
+F 3 "" H 4650 1200 50  0001 C CNN
+	1    4650 1200
+	1    0    0    -1
+$EndComp
+$Comp
+L power:GNDA #PWR?
+U 1 1 601650AC
+P 4150 1700
+AR Path="/5FE332ED/601650AC" Ref="#PWR?"  Part="1"
+AR Path="/5FE3342F/601650AC" Ref="#PWR0104"  Part="1"
+F 0 "#PWR0104" H 4150 1450 50  0001 C CNN
+F 1 "GNDA" H 4155 1527 50  0000 C CNN
+F 2 "" H 4150 1700 50  0001 C CNN
+F 3 "" H 4150 1700 50  0001 C CNN
+	1    4150 1700
+	1    0    0    -1
+$EndComp
+Text GLabel 3150 1400 0    50   Input ~ 0
+Opamp5V
+Text GLabel 2400 2850 1    50   Input ~ 0
+Opamp5V
 $EndSCHEMATC
