File: mixer2.sch (KiCad schematic (older format))
At the start: 24 parts, among them Q1 MMBT5089, U2 SA612, Y1 28.636 MHz

Commit message: Pcb vHA8KDA
Parts:
- C10, C11, C12, C13, C14, C15, C16, C17, C18, C19, C20, C21, C22, C23: footprint Capacitor_SMD:C_0805_2012Metric_Pad1.15x1.40mm_HandSolder -> Capacitor_SMD:C_0805_2012Metric_Pad1.18x1.45mm_HandSolder
- R4, R5, R6, R7, R8: footprint Resistor_SMD:R_0805_2012Metric_Pad1.15x1.40mm_HandSolder -> Resistor_SMD:R_0805_2012Metric_Pad1.20x1.40mm_HandSolder
Changed lines of the file:
@@
 F 0 "C19" H 7215 3246 50  0000 L CNN
 F 1 "10n" H 7215 3155 50  0000 L CNN
-F 2 "Capacitor_SMD:C_0805_2012Metric_Pad1.15x1.40mm_HandSolder" H 7138 3050 50  0001 C CNN
+F 2 "Capacitor_SMD:C_0805_2012Metric_Pad1.18x1.45mm_HandSolder" H 7138 3050 50  0001 C CNN
 F 3 "~" H 7100 3200 50  0001 C CNN
 	1    7100 3200
@@
 F 0 "C20" H 7615 3246 50  0000 L CNN
 F 1 "100n" H 7615 3155 50  0000 L CNN
-F 2 "Capacitor_SMD:C_0805_2012Metric_Pad1.15x1.40mm_HandSolder" H 7538 3050 50  0001 C CNN
+F 2 "Capacitor_SMD:C_0805_2012Metric_Pad1.18x1.45mm_HandSolder" H 7538 3050 50  0001 C CNN
 F 3 "~" H 7500 3200 50  0001 C CNN
 	1    7500 3200
@@
 F 0 "R8" V 7493 3050 50  0000 C CNN
 F 1 "100" V 7584 3050 50  0000 C CNN
-F 2 "Resistor_SMD:R_0805_2012Metric_Pad1.15x1.40mm_HandSolder" V 7630 3050 50  0001 C CNN
+F 2 "Resistor_SMD:R_0805_2012Metric_Pad1.20x1.40mm_HandSolder" V 7630 3050 50  0001 C CNN
 F 3 "~" H 7700 3050 50  0001 C CNN
 	1    7700 3050
@@
 F 0 "C23" H 8065 3246 50  0000 L CNN
 F 1 "100n" H 8065 3155 50  0000 L CNN
-F 2 "Capacitor_SMD:C_0805_2012Metric_Pad1.15x1.40mm_HandSolder" H 7988 3050 50  0001 C CNN
+F 2 "Capacitor_SMD:C_0805_2012Metric_Pad1.18x1.45mm_HandSolder" H 7988 3050 50  0001 C CNN
 F 3 "~" H 7950 3200 50  0001 C CNN
 	1    7950 3200
@@
 F 0 "C18" H 6215 3996 50  0000 L CNN
 F 1 "10n" H 6215 3905 50  0000 L CNN
-F 2 "Capacitor_SMD:C_0805_2012Metric_Pad1.15x1.40mm_HandSolder" H 6138 3800 50  0001 C CNN
+F 2 "Capacitor_SMD:C_0805_2012Metric_Pad1.18x1.45mm_HandSolder" H 6138 3800 50  0001 C CNN
 F 3 "~" H 6100 3950 50  0001 C CNN
 	1    6100 3950
@@
 F 0 "C16" H 5415 3446 50  0000 L CNN
 F 1 "100p" H 5415 3355 50  0000 L CNN
-F 2 "Capacitor_SMD:C_0805_2012Metric_Pad1.15x1.40mm_HandSolder" H 5338 3250 50  0001 C CNN
+F 2 "Capacitor_SMD:C_0805_2012Metric_Pad1.18x1.45mm_HandSolder" H 5338 3250 50  0001 C CNN
 F 3 "~" H 5300 3400 50  0001 C CNN
 	1    5300 3400
@@
 F 0 "C17" V 5498 3700 50  0000 C CNN
 F 1 "10n" V 5589 3700 50  0000 C CNN
-F 2 "Capacitor_SMD:C_0805_2012Metric_Pad1.15x1.40mm_HandSolder" H 5788 3550 50  0001 C CNN
+F 2 "Capacitor_SMD:C_0805_2012Metric_Pad1.18x1.45mm_HandSolder" H 5788 3550 50  0001 C CNN
 F 3 "~" H 5750 3700 50  0001 C CNN
 	1    5750 3700
@@
 F 0 "R7" H 5220 4796 50  0000 L CNN
 F 1 "5k" H 5220 4705 50  0000 L CNN
-F 2 "Resistor_SMD:R_0805_2012Metric_Pad1.15x1.40mm_HandSolder" V 5080 4750 50  0001 C CNN
+F 2 "Resistor_SMD:R_0805_2012Metric_Pad1.20x1.40mm_HandSolder" V 5080 4750 50  0001 C CNN
 F 3 "~" H 5150 4750 50  0001 C CNN
 	1    5150 4750
@@
 F 0 "C15" V 4952 4200 50  0000 C CNN
 F 1 "10n" V 4861 4200 50  0000 C CNN
-F 2 "Capacitor_SMD:C_0805_2012Metric_Pad1.15x1.40mm_HandSolder" H 4738 4050 50  0001 C CNN
+F 2 "Capacitor_SMD:C_0805_2012Metric_Pad1.18x1.45mm_HandSolder" H 4738 4050 50  0001 C CNN
 F 3 "~" H 4700 4200 50  0001 C CNN
 	1    4700 4200
@@
 F 0 "R5" H 3870 3796 50  0000 L CNN
 F 1 "28k" H 3870 3705 50  0000 L CNN
-F 2 "Resistor_SMD:R_0805_2012Metric_Pad1.15x1.40mm_HandSolder" V 3730 3750 50  0001 C CNN
+F 2 "Resistor_SMD:R_0805_2012Metric_Pad1.20x1.40mm_HandSolder" V 3730 3750 50  0001 C CNN
 F 3 "~" H 3800 3750 50  0001 C CNN
 	1    3800 3750
@@
 F 0 "R6" H 3870 4096 50  0000 L CNN
 F 1 "31k" H 3870 4005 50  0000 L CNN
-F 2 "Resistor_SMD:R_0805_2012Metric_Pad1.15x1.40mm_HandSolder" V 3730 4050 50  0001 C CNN
+F 2 "Resistor_SMD:R_0805_2012Metric_Pad1.20x1.40mm_HandSolder" V 3730 4050 50  0001 C CNN
 F 3 "~" H 3800 4050 50  0001 C CNN
 	1    3800 4050
@@
 F 0 "C11" H 3515 4096 50  0000 L CNN
 F 1 "100n" H 3515 4005 50  0000 L CNN
-F 2 "Capacitor_SMD:C_0805_2012Metric_Pad1.15x1.40mm_HandSolder" H 3438 3900 50  0001 C CNN
+F 2 "Capacitor_SMD:C_0805_2012Metric_Pad1.18x1.45mm_HandSolder" H 3438 3900 50  0001 C CNN
 F 3 "~" H 3400 4050 50  0001 C CNN
 	1    3400 4050
@@
 F 0 "C10" H 3115 4096 50  0000 L CNN
 F 1 "10n" H 3115 4005 50  0000 L CNN
-F 2 "Capacitor_SMD:C_0805_2012Metric_Pad1.15x1.40mm_HandSolder" H 3038 3900 50  0001 C CNN
+F 2 "Capacitor_SMD:C_0805_2012Metric_Pad1.18x1.45mm_HandSolder" H 3038 3900 50  0001 C CNN
 F 3 "~" H 3000 4050 50  0001 C CNN
 	1    3000 4050
@@
 F 0 "C21" H 7665 4246 50  0000 L CNN
 F 1 "36p" H 7665 4155 50  0000 L CNN
-F 2 "Capacitor_SMD:C_0805_2012Metric_Pad1.15x1.40mm_HandSolder" H 7588 4050 50  0001 C CNN
+F 2 "Capacitor_SMD:C_0805_2012Metric_Pad1.18x1.45mm_HandSolder" H 7588 4050 50  0001 C CNN
 F 3 "~" H 7550 4200 50  0001 C CNN
 	1    7550 4200
@@
 F 0 "C22" H 7665 4546 50  0000 L CNN
 F 1 "36p" H 7665 4455 50  0000 L CNN
-F 2 "Capacitor_SMD:C_0805_2012Metric_Pad1.15x1.40mm_HandSolder" H 7588 4350 50  0001 C CNN
+F 2 "Capacitor_SMD:C_0805_2012Metric_Pad1.18x1.45mm_HandSolder" H 7588 4350 50  0001 C CNN
 F 3 "~" H 7550 4500 50  0001 C CNN
 	1    7550 4500
@@
 F 0 "C14" H 4515 3096 50  0000 L CNN
 F 1 "10n" H 4515 3005 50  0000 L CNN
-F 2 "Capacitor_SMD:C_0805_2012Metric_Pad1.15x1.40mm_HandSolder" H 4438 2900 50  0001 C CNN
+F 2 "Capacitor_SMD:C_0805_2012Metric_Pad1.18x1.45mm_HandSolder" H 4438 2900 50  0001 C CNN
 F 3 "~" H 4400 3050 50  0001 C CNN
 	1    4400 3050
@@
 F 0 "C13" H 4115 3096 50  0000 L CNN
 F 1 "100n" H 4115 3005 50  0000 L CNN
-F 2 "Capacitor_SMD:C_0805_2012Metric_Pad1.15x1.40mm_HandSolder" H 4038 2900 50  0001 C CNN
+F 2 "Capacitor_SMD:C_0805_2012Metric_Pad1.18x1.45mm_HandSolder" H 4038 2900 50  0001 C CNN
 F 3 "~" H 4000 3050 50  0001 C CNN
 	1    4000 3050
@@
 F 0 "R4" V 3593 2900 50  0000 C CNN
 F 1 "100" V 3684 2900 50  0000 C CNN
-F 2 "Resistor_SMD:R_0805_2012Metric_Pad1.15x1.40mm_HandSolder" V 3730 2900 50  0001 C CNN
+F 2 "Resistor_SMD:R_0805_2012Metric_Pad1.20x1.40mm_HandSolder" V 3730 2900 50  0001 C CNN
 F 3 "~" H 3800 2900 50  0001 C CNN
 	1    3800 2900
@@
 F 0 "C12" H 3665 3096 50  0000 L CNN
 F 1 "100n" H 3665 3005 50  0000 L CNN
-F 2 "Capacitor_SMD:C_0805_2012Metric_Pad1.15x1.40mm_HandSolder" H 3588 2900 50  0001 C CNN
+F 2 "Capacitor_SMD:C_0805_2012Metric_Pad1.18x1.45mm_HandSolder" H 3588 2900 50  0001 C CNN
 F 3 "~" H 3550 3050 50  0001 C CNN
 	1    3550 3050

Commit message: IF1 modified to 37,224 MHz
Parts:
- Y1: value 28.636 MHz -> 28.224 MHz; Farnell 2819267RL -> 2819265
Changed lines of the file:
@@
 P 8050 4550
 F 0 "Y1" V 8004 4681 50  0000 L CNN
-F 1 "28.636 MHz" V 8095 4681 50  0000 L CNN
+F 1 "28.224 MHz" V 8095 4681 50  0000 L CNN
 F 2 "Crystal:Crystal_HC49-U_Vertical" H 8050 4550 50  0001 C CNN
 F 3 "~" H 8050 4550 50  0001 C CNN
-F 4 "2819267RL" V 8200 4900 50  0000 C CNN "Farnell"
+F 4 "2819265" V 8200 4850 50  0000 C CNN "Farnell"
 	1    8050 4550
 	0    1    1    0

Commit message: FPGA change and new project file
Parts:
- renumbered C19 to C?, C20 to C?, C23 to C?, C18 to C?, C16 to C?, C17 to C?, C15 to C?, C11 to C?, C10 to C?, C21 to C?, C22 to C?, C14 to C?, C13 to C?, C12 to C?, L9 to L?, L10 to L?, Q1 to Q?, R8 to R?, R7 to R?, R5 to R?, R6 to R?, R4 to R?, Y1 to Y?

Commit message: PCB is Done... Needs DRC check
Parts:
- gave numbers to parts that had none: 23

Commit message: RX PCB revision: Diff amp + Mixer2
Parts:
- C11, C12, C13: footprint Capacitor_SMD:C_0805_2012Metric_Pad1.18x1.45mm_HandSolder -> Capacitor_SMD:C_0805_2012Metric_Pad1.15x1.40mm_HandSolder
- C14: renamed from C18; footprint Capacitor_SMD:C_0805_2012Metric_Pad1.18x1.45mm_HandSolder -> Capacitor_SMD:C_0805_2012Metric_Pad1.15x1.40mm_HandSolder
- C15: renamed from C19; footprint Capacitor_SMD:C_0805_2012Metric_Pad1.18x1.45mm_HandSolder -> Capacitor_SMD:C_0805_2012Metric_Pad1.15x1.40mm_HandSolder
- C16: renamed from C22; footprint Capacitor_SMD:C_0805_2012Metric_Pad1.18x1.45mm_HandSolder -> Capacitor_SMD:C_0805_2012Metric_Pad1.15x1.40mm_HandSolder
- C17: renamed from C15; footprint Capacitor_SMD:C_0805_2012Metric_Pad1.18x1.45mm_HandSolder -> Capacitor_SMD:C_0805_2012Metric_Pad1.15x1.40mm_HandSolder
- C18: renamed from C16; footprint Capacitor_SMD:C_0805_2012Metric_Pad1.18x1.45mm_HandSolder -> Capacitor_SMD:C_0805_2012Metric_Pad1.15x1.40mm_HandSolder
- C19: renamed from C17; footprint Capacitor_SMD:C_0805_2012Metric_Pad1.18x1.45mm_HandSolder -> Capacitor_SMD:C_0805_2012Metric_Pad1.15x1.40mm_HandSolder
- C20: renamed from C9; footprint Capacitor_SMD:C_0805_2012Metric_Pad1.18x1.45mm_HandSolder -> Capacitor_SMD:C_0805_2012Metric_Pad1.15x1.40mm_HandSolder
- C21: renamed from C10; footprint Capacitor_SMD:C_0805_2012Metric_Pad1.18x1.45mm_HandSolder -> Capacitor_SMD:C_0805_2012Metric_Pad1.15x1.40mm_HandSolder
- C22: renamed from C14; footprint Capacitor_SMD:C_0805_2012Metric_Pad1.18x1.45mm_HandSolder -> Capacitor_SMD:C_0805_2012Metric_Pad1.15x1.40mm_HandSolder
- C23: renamed from C20; footprint Capacitor_SMD:C_0805_2012Metric_Pad1.18x1.45mm_HandSolder -> Capacitor_SMD:C_0805_2012Metric_Pad1.15x1.40mm_HandSolder
- C24: renamed from C21; footprint Capacitor_SMD:C_0805_2012Metric_Pad1.18x1.45mm_HandSolder -> Capacitor_SMD:C_0805_2012Metric_Pad1.15x1.40mm_HandSolder
- R10: renamed from R4; footprint Resistor_SMD:R_0805_2012Metric_Pad1.20x1.40mm_HandSolder -> Resistor_SMD:R_0805_2012Metric_Pad1.15x1.40mm_HandSolder
- R11: renamed from R8; footprint Resistor_SMD:R_0805_2012Metric_Pad1.20x1.40mm_HandSolder -> Resistor_SMD:R_0805_2012Metric_Pad1.15x1.40mm_HandSolder
- R12: renamed from R5; footprint Resistor_SMD:R_0805_2012Metric_Pad1.20x1.40mm_HandSolder -> Resistor_SMD:R_0805_2012Metric_Pad1.15x1.40mm_HandSolder
- R13: renamed from R6; footprint Resistor_SMD:R_0805_2012Metric_Pad1.20x1.40mm_HandSolder -> Resistor_SMD:R_0805_2012Metric_Pad1.15x1.40mm_HandSolder
- R14: renamed from R7; footprint Resistor_SMD:R_0805_2012Metric_Pad1.20x1.40mm_HandSolder -> Resistor_SMD:R_0805_2012Metric_Pad1.15x1.40mm_HandSolder
