File: receiver_test.kicad_pcb (KiCad board)
At the start: 2 copper layers, 12 parts, among them J1 Conn_Coaxial, Q1 MMBT5089, U1 ADE-1H+, U2 SA612, U3 MCP6D11

Commit message: majdnem kész a nyák béta verziója
Parts:
- added C10: 10n, Capacitor_SMD:C_0805_2012Metric_Pad1.15x1.40mm_HandSolder, F.Cu at (171.2, 73.2)
- added C11: 100n, Capacitor_SMD:C_0805_2012Metric_Pad1.15x1.40mm_HandSolder, F.Cu at (176.3, 73.2)
- added C12: 100n, Capacitor_SMD:C_0805_2012Metric_Pad1.15x1.40mm_HandSolder, F.Cu at (163.6, 73.1)
- added C13: 100n, Capacitor_SMD:C_0805_2012Metric_Pad1.15x1.40mm_HandSolder, F.Cu at (166.1, 73.2)
- added C14: 10n, Capacitor_SMD:C_0805_2012Metric_Pad1.15x1.40mm_HandSolder, F.Cu at (168.7, 73.2)
- added C15: 10n, Capacitor_SMD:C_0805_2012Metric_Pad1.15x1.40mm_HandSolder, F.Cu at (174.8, 64.0)
- added C16: 100p, Capacitor_SMD:C_0805_2012Metric_Pad1.15x1.40mm_HandSolder, F.Cu at (169.2, 67.1)
- added C17: 10n, Capacitor_SMD:C_0805_2012Metric_Pad1.15x1.40mm_HandSolder, F.Cu at (164.6, 67.1)
- added C18: 10n, Capacitor_SMD:C_0805_2012Metric_Pad1.15x1.40mm_HandSolder, F.Cu at (173.7, 58.4)
- added C19: 10n, Capacitor_SMD:C_0805_2012Metric_Pad1.15x1.40mm_HandSolder, F.Cu at (163.1, 63.5)
- added C20: 100n, Capacitor_SMD:C_0805_2012Metric_Pad1.15x1.40mm_HandSolder, F.Cu at (165.6, 63.5)
- added C21: 36p, Capacitor_SMD:C_0805_2012Metric_Pad1.15x1.40mm_HandSolder, F.Cu at (162.1, 58.4)
- added C22: 36p, Capacitor_SMD:C_0805_2012Metric_Pad1.15x1.40mm_HandSolder, F.Cu at (162.1, 54.3)
- added C23: 100n, Capacitor_SMD:C_0805_2012Metric_Pad1.15x1.40mm_HandSolder, F.Cu at (161.0, 73.1)
- added C24: 68p, Capacitor_SMD:C_0805_2012Metric_Pad1.15x1.40mm_HandSolder, F.Cu at (184.9, 52.3)
- added C25: 15p, Capacitor_SMD:C_0805_2012Metric_Pad1.15x1.40mm_HandSolder, F.Cu at (182.4, 52.3)
- added C26: 470p, Capacitor_SMD:C_0805_2012Metric_Pad1.15x1.40mm_HandSolder, F.Cu at (187.5, 52.3)
- added C27: 18p, Capacitor_SMD:C_0805_2012Metric_Pad1.15x1.40mm_HandSolder, F.Cu at (177.8, 58.9)
- added C28: 18p, Capacitor_SMD:C_0805_2012Metric_Pad1.15x1.40mm_HandSolder, F.Cu at (190.0, 52.3)
- added C29: 180p, Capacitor_SMD:C_0805_2012Metric_Pad1.15x1.40mm_HandSolder, F.Cu at (180.3, 63.0)
- added C30: 180p, Capacitor_SMD:C_0805_2012Metric_Pad1.15x1.40mm_HandSolder, F.Cu at (190.0, 60.5)
- added C31: 9p, Capacitor_SMD:C_0805_2012Metric_Pad1.15x1.40mm_HandSolder, F.Cu at (212.9, 60.0)
- added C32: 10n, Capacitor_SMD:C_0805_2012Metric_Pad1.15x1.40mm_HandSolder, F.Cu at (219.0, 59.9)
- added C33: 47u, Capacitor_SMD:CP_Elec_6.3x5.3, F.Cu at (162.1, 105.4)
- added C34: 100n, Capacitor_SMD:C_0805_2012Metric_Pad1.15x1.40mm_HandSolder, F.Cu at (167.1, 105.1)
- added C35: 10p, Capacitor_SMD:C_0805_2012Metric_Pad1.15x1.40mm_HandSolder, F.Cu at (195.6, 71.1)
- added C36: 10n, Capacitor_SMD:C_0805_2012Metric_Pad1.15x1.40mm_HandSolder, F.Cu at (207.8, 59.9)
- added C37: 100n, Capacitor_SMD:C_0805_2012Metric_Pad1.15x1.40mm_HandSolder, F.Cu at (207.8, 57.4)
- added C38: 100n, Capacitor_SMD:C_0805_2012Metric_Pad1.15x1.40mm_HandSolder, F.Cu at (210.8, 65.5)
- added C39: 33p, Capacitor_SMD:C_0805_2012Metric_Pad1.15x1.40mm_HandSolder, F.Cu at (180.3, 65.2)
- added C40: 33p, Capacitor_SMD:C_0805_2012Metric_Pad1.15x1.40mm_HandSolder, F.Cu at (186.9, 60.5)
- added C5: 8p2, Capacitor_SMD:C_0805_2012Metric_Pad1.15x1.40mm_HandSolder, F.Cu at (116.2, 75.9)
- added C6: 43p, Capacitor_SMD:C_0805_2012Metric_Pad1.15x1.40mm_HandSolder, F.Cu at (116.2, 72.9)
- added C7: 51p, Capacitor_SMD:C_0805_2012Metric_Pad1.15x1.40mm_HandSolder, F.Cu at (125.7, 72.9)
- added C8: 3p3, Capacitor_SMD:C_0805_2012Metric_Pad1.15x1.40mm_HandSolder, F.Cu at (121.0, 75.9)
- added C9: 1n, Capacitor_SMD:C_0805_2012Metric_Pad1.15x1.40mm_HandSolder, F.Cu at (119.9, 68.6)
- added D1: Red, LED_SMD:LED_0805_2012Metric_Pad1.15x1.40mm_HandSolder, F.Cu at (172.2, 105.1)
- added H2: 3mm spacer, MountingHole:MountingHole_3.2mm_M3, F.Cu at (90.7, 26.6)
- added H3: 3mm spacer, MountingHole:MountingHole_3.2mm_M3, F.Cu at (98.7, 18.6)
- added H4: 3mm spacer, MountingHole:MountingHole_3.2mm_M3, F.Cu at (98.7, 26.6)
- added J2: IF_IN, Connector_Coaxial:SMA_Molex_73251-1153_EdgeMount_Horizontal, F.Cu at (34.5, 171.1)
- added J3: Conn_01x02_Male, Connector_PinSocket_2.54mm:PinSocket_1x02_P2.54mm_Vertical, F.Cu at (209.8, 91.4)
- added J4: Conn_01x02_Male, Connector_PinSocket_2.54mm:PinSocket_1x02_P2.54mm_Vertical, F.Cu at (209.8, 87.4)
- added J6: 5V, Connector_PinSocket_2.54mm:PinSocket_1x02_P2.54mm_Vertical, F.Cu at (156.5, 106.7)
- added L10: 2u2, Inductor_SMD:L_0805_2012Metric_Pad1.15x1.40mm_HandSolder, F.Cu at (178.8, 69.1)
- added L11: 2u2, Inductor_SMD:L_0805_2012Metric_Pad1.15x1.40mm_HandSolder, F.Cu at (177.8, 55.9)
- added L12: 2u2, Inductor_SMD:L_0805_2012Metric_Pad1.15x1.40mm_HandSolder, F.Cu at (183.4, 49.3)
- added L13: 10u, Inductor_SMD:L_1210_3225Metric_Pad1.42x2.65mm_HandSolder, F.Cu at (182.9, 59.4)
- added L14: 10u, Inductor_SMD:L_1210_3225Metric_Pad1.42x2.65mm_HandSolder, F.Cu at (188.4, 56.4)
- added L15: 2u2, Inductor_SMD:L_0805_2012Metric_Pad1.15x1.40mm_HandSolder, F.Cu at (183.4, 55.9)
- added L16: 220n, Inductor_SMD:L_1210_3225Metric_Pad1.42x2.65mm_HandSolder, F.Cu at (185.4, 65.5)
- added L17: 220n, Inductor_SMD:L_1210_3225Metric_Pad1.42x2.65mm_HandSolder, F.Cu at (189.5, 65.5)
- added L18: 8u2, Inductor_SMD:L_1210_3225Metric_Pad1.42x2.65mm_HandSolder, F.Cu at (212.9, 55.9)
- added L19: 8u2, Inductor_SMD:L_1210_3225Metric_Pad1.42x2.65mm_HandSolder, F.Cu at (214.9, 64.0)
- added L4: 2u2, Inductor_SMD:L_0805_2012Metric_Pad1.15x1.40mm_HandSolder, F.Cu at (119.1, 42.6)
- added L5: 330n, Inductor_SMD:L_1210_3225Metric_Pad1.42x2.65mm_HandSolder, F.Cu at (113.8, 40.3)
- added L6: 470n, Inductor_SMD:L_0805_2012Metric_Pad1.15x1.40mm_HandSolder, F.Cu at (122.9, 35.6)
- added L9: 180n, Inductor_SMD:L_1210_3225Metric_Pad1.42x2.65mm_HandSolder, F.Cu at (170.1, 63.5)
- added Q2: BC847BS, Package_TO_SOT_SMD:SOT-363_SC-70-6, F.Cu at (215.4, 59.9)
- added R1: nk, Resistor_SMD:R_0805_2012Metric_Pad1.15x1.40mm_HandSolder, F.Cu at (199.6, 78.2)
- added R10: 1.2k, Resistor_SMD:R_0805_2012Metric_Pad1.15x1.40mm_HandSolder, F.Cu at (221.0, 54.9)
- added R11: 470, Resistor_SMD:R_0805_2012Metric_Pad1.15x1.40mm_HandSolder, F.Cu at (169.7, 105.2)
- added R12: BP, Resistor_SMD:R_1206_3216Metric_Pad1.42x1.75mm_HandSolder, F.Cu at (207.3, 44.7)
- added R13: 2k5, Resistor_SMD:R_0805_2012Metric_Pad1.15x1.40mm_HandSolder, F.Cu at (193.5, 72.7)
- added R14: 19k, Resistor_SMD:R_0805_2012Metric_Pad1.15x1.40mm_HandSolder, F.Cu at (214.9, 67.1)
- added R15: 31k, Resistor_SMD:R_0805_2012Metric_Pad1.15x1.40mm_HandSolder, F.Cu at (218.9, 57.4)
- added R16: 27, Resistor_SMD:R_0805_2012Metric_Pad1.15x1.40mm_HandSolder, F.Cu at (191.5, 83.8)
- added R17: 39, Resistor_SMD:R_0805_2012Metric_Pad1.15x1.40mm_HandSolder, F.Cu at (191.5, 81.8)
- added R18: 47, Resistor_SMD:R_0805_2012Metric_Pad1.15x1.40mm_HandSolder, F.Cu at (191.5, 79.8)
- added R19: 33, Resistor_SMD:R_0805_2012Metric_Pad1.15x1.40mm_HandSolder, F.Cu at (191.5, 86.4)
- added R2: nk, Resistor_SMD:R_0805_2012Metric_Pad1.15x1.40mm_HandSolder, F.Cu at (197.1, 78.2)
- added R20: 10, Resistor_SMD:R_0805_2012Metric_Pad1.15x1.40mm_HandSolder, F.Cu at (188.5, 80.8)
- added R21: 3, Resistor_SMD:R_0805_2012Metric_Pad1.15x1.40mm_HandSolder, F.Cu at (205.2, 79.8)
- added R22: 27, Resistor_SMD:R_0805_2012Metric_Pad1.15x1.40mm_HandSolder, F.Cu at (205.2, 85.9)
- added R23: 39, Resistor_SMD:R_0805_2012Metric_Pad1.15x1.40mm_HandSolder, F.Cu at (205.2, 83.8)
- added R24: 47, Resistor_SMD:R_0805_2012Metric_Pad1.15x1.40mm_HandSolder, F.Cu at (205.2, 81.8)
- added R25: 100, Resistor_SMD:R_0805_2012Metric_Pad1.15x1.40mm_HandSolder, F.Cu at (208.8, 63.5)
- added R26: BP, Resistor_SMD:R_1206_3216Metric_Pad1.42x1.75mm_HandSolder, F.Cu at (187.5, 90.9)
- added R27: BP, Resistor_SMD:R_1206_3216Metric_Pad1.42x1.75mm_HandSolder, F.Cu at (201.7, 91.0)
- added R28: BP, Resistor_SMD:R_1206_3216Metric_Pad1.42x1.75mm_HandSolder, F.Cu at (186.9, 72.1)
- added R29: BP, Resistor_SMD:R_1206_3216Metric_Pad1.42x1.75mm_HandSolder, F.Cu at (54.9, 169.7)
- added R3: 10k, Resistor_SMD:R_0805_2012Metric_Pad1.15x1.40mm_HandSolder, F.Cu at (198.1, 71.1)
- added R30: BP, Resistor_SMD:R_1206_3216Metric_Pad1.42x1.75mm_HandSolder, F.Cu at (168.2, 49.3)
- added R31: BP, Resistor_SMD:R_1206_3216Metric_Pad1.42x1.75mm_HandSolder, F.Cu at (168.2, 46.2)
- added R32: BP, Resistor_SMD:R_1206_3216Metric_Pad1.42x1.75mm_HandSolder, F.Cu at (195.6, 45.7)
- added R33: BP, Resistor_SMD:R_1206_3216Metric_Pad1.42x1.75mm_HandSolder, F.Cu at (195.6, 48.8)
- added R34: BP, Resistor_SMD:R_1206_3216Metric_Pad1.42x1.75mm_HandSolder, F.Cu at (190.5, 72.1)
- added R35: BP, Resistor_SMD:R_1206_3216Metric_Pad1.42x1.75mm_HandSolder, F.Cu at (215.9, 49.8)
- added R36: BP, Resistor_SMD:R_1206_3216Metric_Pad1.42x1.75mm_HandSolder, F.Cu at (207.3, 51.3)
- added R37: BP, Resistor_SMD:R_1206_3216Metric_Pad1.42x1.75mm_HandSolder, F.Cu at (207.2, 47.8)
- added R38: BP, Resistor_SMD:R_1206_3216Metric_Pad1.42x1.75mm_HandSolder, F.Cu at (206.8, 70.1)
- added R39: BP, Resistor_SMD:R_1206_3216Metric_Pad1.42x1.75mm_HandSolder, F.Cu at (206.8, 74.2)
- added R4: 100, Resistor_SMD:R_0805_2012Metric_Pad1.15x1.40mm_HandSolder, F.Cu at (164.6, 69.6)
- added R40: BP, Resistor_SMD:R_1206_3216Metric_Pad1.42x1.75mm_HandSolder, F.Cu at (224.5, 52.3)
- added R41: BP, Resistor_SMD:R_1206_3216Metric_Pad1.42x1.75mm_HandSolder, F.Cu at (212.9, 70.1)
- added R5: 28k, Resistor_SMD:R_0805_2012Metric_Pad1.15x1.40mm_HandSolder, F.Cu at (169.2, 69.6)
- added R6: 31k, Resistor_SMD:R_0805_2012Metric_Pad1.15x1.40mm_HandSolder, F.Cu at (173.7, 73.1)
- added R7: 5k, Resistor_SMD:R_0805_2012Metric_Pad1.15x1.40mm_HandSolder, F.Cu at (178.8, 73.2)
- added R8: 100, Resistor_SMD:R_0805_2012Metric_Pad1.15x1.40mm_HandSolder, F.Cu at (161.0, 65.0)
- added R9: 1.2k, Resistor_SMD:R_0805_2012Metric_Pad1.15x1.40mm_HandSolder, F.Cu at (213.4, 45.7)
- added TP1: TestPoint, Connector_PinHeader_2.54mm:PinHeader_1x01_P2.54mm_Vertical, F.Cu at (182.9, 84.8)
- added TP10: TestPoint, Connector_PinHeader_2.54mm:PinHeader_1x01_P2.54mm_Vertical, F.Cu at (120.4, 57.9)
- added TP11: TestPoint_2Pole, Connector_PinHeader_2.54mm:PinHeader_1x02_P2.54mm_Vertical, F.Cu at (197.1, 52.8)
- added TP12: TestPoint_2Pole, Connector_PinHeader_2.54mm:PinHeader_1x02_P2.54mm_Vertical, F.Cu at (201.7, 50.8)
- added TP13: TestPoint_2Pole, Connector_PinHeader_2.54mm:PinHeader_1x02_P2.54mm_Vertical, F.Cu at (201.2, 70.6)
- added TP2: TestPoint, Connector_PinHeader_2.54mm:PinHeader_1x01_P2.54mm_Vertical, F.Cu at (193.5, 90.9)
- added TP3: TestPoint, Connector_PinHeader_2.54mm:PinHeader_1x01_P2.54mm_Vertical, F.Cu at (198.1, 90.9)
- added TP4: TestPoint, Connector_PinHeader_2.54mm:PinHeader_1x01_P2.54mm_Vertical, F.Cu at (50.8, 166.6)
- added TP5: TestPoint, Connector_PinHeader_2.54mm:PinHeader_1x01_P2.54mm_Vertical, F.Cu at (182.9, 73.2)
- added TP6: TestPoint, Connector_PinHeader_2.54mm:PinHeader_1x01_P2.54mm_Vertical, F.Cu at (50.8, 170.7)
- added TP7: TestPoint, Connector_PinHeader_2.54mm:PinHeader_1x01_P2.54mm_Vertical, F.Cu at (105.0, 31.4)
- added TP8: TestPoint_2Pole, Connector_PinHeader_2.54mm:PinHeader_1x02_P2.54mm_Vertical, F.Cu at (169.7, 52.8)
- added TP9: TestPoint_2Pole, Connector_PinHeader_2.54mm:PinHeader_1x02_P2.54mm_Vertical, F.Cu at (176.8, 52.8)
- added U4: FST3253, Package_SO:TSSOP-16_4.4x5mm_P0.65mm, F.Cu at (198.6, 83.3)
- added Y1: 28.636 MHz, Crystal:Crystal_HC49-U_Vertical, F.Cu at (157.5, 59.4)
- J1: value Conn_Coaxial -> RF_IN
- L1, L2, L3: footprint Inductor_SMD:L_1206_3216Metric_Pad1.22x1.90mm_HandSolder -> Inductor_SMD:L_1206_3216Metric_Pad1.42x1.75mm_HandSolder
- moved U1 125.2 mm to (43.2, 169.9), turned to 180 degrees
- moved U3 124.3 mm to (221.0, 47.8), turned to 90 degrees
- moved C1 103.6 mm to (165.3, 87.8)
- moved C4 103.6 mm to (178.9, 87.8)
- moved L1 103.6 mm to (166.8, 84.5)
- moved L3 103.6 mm to (177.2, 84.5)
- moved C2 103.6 mm to (168.5, 87.8)
- moved C3 103.6 mm to (173.7, 87.8)
- moved L2 103.6 mm to (172.0, 84.5)
- moved J1 102.2 mm to (160.2, 84.1)
- moved Q1 87.8 mm to (174.8, 69.1), turned to 90 degrees
- moved U2 77.2 mm to (168.1, 58.4), turned to 180 degrees
Connections:
- net /Attenuator/IN renamed /30MHz LPF/OUT
- Q1 pad 1: (no net) -> Net-(C10-Pad1)
- Q1 pad 2: (no net) -> Net-(C15-Pad2)
- Q1 pad 3: (no net) -> Net-(C16-Pad2)
- U1 pad 2: (no net) -> Net-(R29-Pad2)
- U1 pad 3: (no net) -> Net-(R27-Pad1)
- U1 pad 6: (no net) -> Net-(J2-Pad1)
- U2 pad 1: (no net) -> Net-(C17-Pad1)
- U2 pad 2: (no net) -> Net-(C18-Pad1)
- U2 pad 4: (no net) -> /37.4 MHz Amp, and 2nd mixer/out_p
- U2 pad 5: (no net) -> /37.4 MHz Amp, and 2nd mixer/out_n
- U2 pad 6: (no net) -> Net-(C21-Pad2)
- U2 pad 7: (no net) -> Net-(C21-Pad1)
- U2 pad 8: (no net) -> Net-(C19-Pad1)
- U3 pad 1: (no net) -> Net-(R10-Pad2)
- U3 pad 2: (no net) -> /Sheet5FE3342E/DC_CM
- U3 pad 4: (no net) -> Net-(R40-Pad2)
- U3 pad 5: (no net) -> Net-(R10-Pad1)
- U3 pad 6: (no net) -> GND
- U3 pad 8: (no net) -> Net-(R12-Pad1)
Routing:
- net +5VA: track 0.00 -> 139.5 mm, vias 0 -> 6
- net GNDA: track 0.00 -> 99.2 mm, vias 0 -> 13
- net /Sheet5FE3342E/Out+: track 0.00 -> 77.7 mm
- net /Sheet5FE3342E/DC_CM: track 0.00 -> 51.3 mm
- net Net-(R17-Pad1): track 0.00 -> 42.0 mm
- net Net-(C31-Pad2): track 0.00 -> 39.1 mm
- net /Sheet5FE333A0/Out+: track 0.00 -> 36.7 mm
- net Net-(R16-Pad1): track 0.00 -> 33.9 mm
- net Net-(C31-Pad1): track 0.00 -> 27.8 mm
- net /Attenuator/ATT_SEL0: track 0.00 -> 26.3 mm, vias 0 -> 1
- net /Sheet5FE3342E/In+: track 0.00 -> 25.4 mm
- net /Sheet5FE333A0/In-: track 0.00 -> 21.9 mm
- net /Sheet5FE333A0/In+: track 0.00 -> 21.6 mm
- net /Sheet5FE333A0/Out-: track 0.00 -> 21.0 mm
- net Net-(C16-Pad2): track 0.00 -> 20.6 mm
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- added copper zone on B.Cu, net GNDA
Other:
- board outline added: 99.6 x 99.6 mm
- board text added: "Attenuator"
- board text added: "Input LPF"
- board text added: "Power"

Commit message: Footprint reassociation, pcb clear
Parts:
- removed C10, C14, C15, C17, C18, C19, C32, C36: 10n, Capacitor_SMD:C_0805_2012Metric_Pad1.15x1.40mm_HandSolder
- removed C11, C12, C13, C20, C23, C34, C37, C38: 100n, Capacitor_SMD:C_0805_2012Metric_Pad1.15x1.40mm_HandSolder
- removed C16: 100p, Capacitor_SMD:C_0805_2012Metric_Pad1.15x1.40mm_HandSolder
- removed C21, C22: 36p, Capacitor_SMD:C_0805_2012Metric_Pad1.15x1.40mm_HandSolder
- removed C24: 68p, Capacitor_SMD:C_0805_2012Metric_Pad1.15x1.40mm_HandSolder
- removed C25: 15p, Capacitor_SMD:C_0805_2012Metric_Pad1.15x1.40mm_HandSolder
- removed C26: 470p, Capacitor_SMD:C_0805_2012Metric_Pad1.15x1.40mm_HandSolder
- removed C27, C28: 18p, Capacitor_SMD:C_0805_2012Metric_Pad1.15x1.40mm_HandSolder
- removed C29, C30: 180p, Capacitor_SMD:C_0805_2012Metric_Pad1.15x1.40mm_HandSolder
- removed C31: 9p, Capacitor_SMD:C_0805_2012Metric_Pad1.15x1.40mm_HandSolder
- removed C39, C40: 33p, Capacitor_SMD:C_0805_2012Metric_Pad1.15x1.40mm_HandSolder
- removed C9: 1n, Capacitor_SMD:C_0805_2012Metric_Pad1.15x1.40mm_HandSolder
- removed R1, R2: nk, Resistor_SMD:R_0805_2012Metric_Pad1.15x1.40mm_HandSolder
- removed R10, R9: 1.2k, Resistor_SMD:R_0805_2012Metric_Pad1.15x1.40mm_HandSolder
- removed R11: 470, Resistor_SMD:R_0805_2012Metric_Pad1.15x1.40mm_HandSolder
- removed R12, R26, R27, R28, R29, R30, R31, R32, R33, R34, R35, R36, R37, R38, R39, R40, R41: BP, Resistor_SMD:R_1206_3216Metric_Pad1.42x1.75mm_HandSolder
- removed R13: 2k5, Resistor_SMD:R_0805_2012Metric_Pad1.15x1.40mm_HandSolder
- removed R14: 19k, Resistor_SMD:R_0805_2012Metric_Pad1.15x1.40mm_HandSolder
- removed R15, R6: 31k, Resistor_SMD:R_0805_2012Metric_Pad1.15x1.40mm_HandSolder
- removed R16, R22: 27, Resistor_SMD:R_0805_2012Metric_Pad1.15x1.40mm_HandSolder
- removed R17, R23: 39, Resistor_SMD:R_0805_2012Metric_Pad1.15x1.40mm_HandSolder
- removed R18, R24: 47, Resistor_SMD:R_0805_2012Metric_Pad1.15x1.40mm_HandSolder
- removed R19: 33, Resistor_SMD:R_0805_2012Metric_Pad1.15x1.40mm_HandSolder
- removed R20: 10, Resistor_SMD:R_0805_2012Metric_Pad1.15x1.40mm_HandSolder
- removed R21: 3, Resistor_SMD:R_0805_2012Metric_Pad1.15x1.40mm_HandSolder
- removed R25, R4, R8: 100, Resistor_SMD:R_0805_2012Metric_Pad1.15x1.40mm_HandSolder
- removed R3: 10k, Resistor_SMD:R_0805_2012Metric_Pad1.15x1.40mm_HandSolder
- removed R5: 28k, Resistor_SMD:R_0805_2012Metric_Pad1.15x1.40mm_HandSolder
- removed R7: 5k, Resistor_SMD:R_0805_2012Metric_Pad1.15x1.40mm_HandSolder
- added H1: 3mm spacer, MountingHole:MountingHole_3.2mm_M3, F.Cu at (40.2, 163.1)
- added L7: 47n, Inductor_SMD:L_0603_1608Metric_Pad1.05x0.95mm_HandSolder, F.Cu at (48.0, 184.2)
- C35: footprint Capacitor_SMD:C_0805_2012Metric_Pad1.15x1.40mm_HandSolder -> Capacitor_SMD:C_0805_2012Metric_Pad1.18x1.45mm_HandSolder
- C5: value 8p2 -> 390p; footprint Capacitor_SMD:C_0805_2012Metric_Pad1.15x1.40mm_HandSolder -> Capacitor_SMD:C_0805_2012Metric_Pad1.18x1.45mm_HandSolder
- C6: value 43p -> 390p; footprint Capacitor_SMD:C_0805_2012Metric_Pad1.15x1.40mm_HandSolder -> Capacitor_SMD:C_0805_2012Metric_Pad1.18x1.45mm_HandSolder
- C7: value 51p -> 470p; footprint Capacitor_SMD:C_0805_2012Metric_Pad1.15x1.40mm_HandSolder -> Capacitor_SMD:C_0805_2012Metric_Pad1.18x1.45mm_HandSolder
- C8: value 3p3 -> 390p; footprint Capacitor_SMD:C_0805_2012Metric_Pad1.15x1.40mm_HandSolder -> Capacitor_SMD:C_0805_2012Metric_Pad1.18x1.45mm_HandSolder
- L4: value 2u2 -> 47n; footprint Inductor_SMD:L_0805_2012Metric_Pad1.15x1.40mm_HandSolder -> Inductor_SMD:L_0603_1608Metric_Pad1.05x0.95mm_HandSolder
- L5: value 330n -> 39n; footprint Inductor_SMD:L_1210_3225Metric_Pad1.42x2.65mm_HandSolder -> Inductor_SMD:L_0402_1005Metric_Pad0.77x0.64mm_HandSolder
- L6: value 470n -> 47n; footprint Inductor_SMD:L_0805_2012Metric_Pad1.15x1.40mm_HandSolder -> Inductor_SMD:L_0603_1608Metric_Pad1.05x0.95mm_HandSolder
- moved L17 197.2 mm to (28.3, 179.0), turned to 0 degrees
- moved L14 197.0 mm to (34.2, 179.0)
- moved L16 196.3 mm to (28.3, 183.2), turned to 0 degrees
- moved L12 195.2 mm to (39.6, 181.3), turned to 0 degrees
- moved C35 194.9 mm to (27.7, 170.1), turned to 0 degrees
- moved L13 193.5 mm to (34.2, 183.2), turned to 0 degrees
- moved L15 188.9 mm to (39.6, 178.4)
- moved L11 188.7 mm to (39.6, 184.3), turned to 0 degrees
- moved TP12 185.8 mm to (54.5, 164.1), turned to 0 degrees
- moved U3 181.4 mm to (81.7, 164.0), turned to 0 degrees
- moved TP1 173.3 mm to (32.4, 170.9)
- moved TP9 171.5 mm to (46.5, 164.3), turned to 0 degrees
- moved TP5 170.7 mm to (43.4, 171.5)
- moved L19 169.8 mm to (81.0, 168.4)
- moved Q2 168.6 mm to (86.1, 168.2), turned to 0 degrees
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Connections:
- net /37.4 MHz Amp, and 2nd mixer/out_n renamed /37.4 MHz Amp, and 2nd mixer/Out-
- net /37.4 MHz Amp, and 2nd mixer/out_p renamed /37.4 MHz Amp, and 2nd mixer/Out+
- C5 pad 1: Net-(C5-Pad1) -> /37.4 MHz BPF/IN
- C5 pad 2: /37.4 MHz Inv-Chebysev BPF/IN -> GNDA
- C6 pad 1: Net-(C6-Pad1) -> /37.4 MHz BPF/IN
- C7 pad 1: Net-(C7-Pad1) -> Net-(C6-Pad2)
- C7 pad 2: Net-(C6-Pad2) -> /37.4 MHz BPF/OUT
- C8 pad 1: Net-(C8-Pad1) -> /37.4 MHz BPF/OUT
- C8 pad 2: Net-(C6-Pad2) -> GNDA
- D1 pad 2: Net-(D1-Pad2) -> (no net)
- L10 pad 2: Net-(L10-Pad2) -> (no net)
- L11 pad 1: Net-(C26-Pad1) -> /Sheet5FE333A0/In+
- L11 pad 2: /Sheet5FE333A0/In+ -> (no net)
- L12 pad 1: Net-(C26-Pad2) -> /Sheet5FE333A0/In-
- L12 pad 2: /Sheet5FE333A0/In- -> (no net)
- L13 pad 1: Net-(C29-Pad2) -> (no net)
- L13 pad 2: Net-(C27-Pad1) -> Net-(C29-Pad2)
- L14 pad 1: Net-(C30-Pad1) -> (no net)
- L14 pad 2: Net-(C28-Pad1) -> Net-(C30-Pad1)
- L4 pad 1: Net-(C6-Pad2) -> /37.4 MHz BPF/IN
- L4 pad 2: Net-(C5-Pad1) -> GNDA
- L5 pad 1: Net-(C6-Pad1) -> /37.4 MHz BPF/IN
- L5 pad 2: GND -> Net-(C6-Pad2)
- L6 pad 1: Net-(C7-Pad1) -> Net-(C6-Pad2)
- L6 pad 2: GND -> /37.4 MHz BPF/OUT
- L9 pad 1: Net-(C13-Pad1) -> (no net)
- Q1 pad 1: Net-(C10-Pad1) -> (no net)
- Q2 pad 1: Net-(Q2-Pad1) -> (no net)
- Q2 pad 4: Net-(Q2-Pad4) -> (no net)
- TP10 pad 1: /37.4 MHz Inv-Chebysev BPF/OUT -> /37.4 MHz BPF/OUT
- TP12 pad 1: /Sheet5FE3342E/In+ -> (no net)
- TP12 pad 2: /Sheet5FE3342E/In- -> (no net)
- TP5 pad 1: /37.4 MHz Amp, and 2nd mixer/IN -> (no net)
- TP7 pad 1: /37.4 MHz Inv-Chebysev BPF/IN -> /37.4 MHz BPF/IN
- U2 pad 1: Net-(C17-Pad1) -> (no net)
- U2 pad 2: Net-(C18-Pad1) -> (no net)
- U2 pad 6: Net-(C21-Pad2) -> (no net)
- U2 pad 8: Net-(C19-Pad1) -> (no net)
- U3 pad 1: Net-(R10-Pad2) -> (no net)
- U3 pad 2: /Sheet5FE3342E/DC_CM -> (no net)
- U3 pad 4: Net-(R40-Pad2) -> (no net)
- U3 pad 5: Net-(R10-Pad1) -> (no net)
- U3 pad 6: GND -> (no net)
- U3 pad 8: Net-(R12-Pad1) -> (no net)
- U4 pad 11: /Attenuator/10dB_out -> (no net)
- U4 pad 12: /Attenuator/20dB_out -> (no net)
- U4 pad 13: /Attenuator/30dB_out -> (no net)
- U4 pad 3: /Attenuator/30dB_in -> (no net)
- U4 pad 4: /Attenuator/20dB_in -> (no net)
- U4 pad 5: /Attenuator/10dB_in -> (no net)
Routing:
- net +5VA: track 139.5 -> 0.00 mm, vias 6 -> 0
- net /Sheet5FE3342E/Out+: track 77.7 -> 0.00 mm
- net GNDA: track 99.2 -> 23.9 mm, vias 13 -> 0
- net /Sheet5FE3342E/DC_CM: track 51.3 -> 0.00 mm
- net Net-(R17-Pad1): track 42.0 -> 0.00 mm
- net Net-(C31-Pad2): track 39.1 -> 0.00 mm
- net /Sheet5FE333A0/Out+: track 36.7 -> 0.00 mm
- net Net-(R16-Pad1): track 33.9 -> 0.00 mm
- net Net-(C31-Pad1): track 27.8 -> 0.00 mm
- net /Attenuator/ATT_SEL0: track 26.3 -> 0.00 mm, vias 1 -> 0
- net /Sheet5FE3342E/In+: track 25.4 -> 0.00 mm
- net /Sheet5FE333A0/In-: track 21.9 -> 0.00 mm
- net /Sheet5FE333A0/In+: track 21.6 -> 0.00 mm
- net /Sheet5FE333A0/Out-: track 21.0 -> 0.00 mm
- net Net-(C16-Pad2): track 20.6 -> 0.00 mm
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- removed copper zone on B.Cu, net GNDA
Other:
- board outline removed
- board text removed: "Attenuator"
- board text removed: "Input LPF"
- board text removed: "Power"

Commit message: Pcb vHA8KDA
Parts:
- added C10: 10n, Capacitor_SMD:C_0805_2012Metric_Pad1.18x1.45mm_HandSolder, F.Cu at (75.6, 97.9)
- added C11: 100n, Capacitor_SMD:C_0805_2012Metric_Pad1.18x1.45mm_HandSolder, F.Cu at (74.9, 96.1)
- added C12: 100n, Capacitor_SMD:C_0805_2012Metric_Pad1.18x1.45mm_HandSolder, F.Cu at (71.3, 89.6)
- added C13: 100n, Capacitor_SMD:C_0805_2012Metric_Pad1.18x1.45mm_HandSolder, F.Cu at (74.4, 90.6)
- added C14: 10n, Capacitor_SMD:C_0805_2012Metric_Pad1.18x1.45mm_HandSolder, F.Cu at (74.3, 88.6)
- added C15: 10n, Capacitor_SMD:C_0805_2012Metric_Pad1.18x1.45mm_HandSolder, F.Cu at (74.9, 101.8)
- added C16: 100p, Capacitor_SMD:C_0805_2012Metric_Pad1.18x1.45mm_HandSolder, F.Cu at (81.8, 96.6)
- added C17: 10n, Capacitor_SMD:C_0805_2012Metric_Pad1.18x1.45mm_HandSolder, F.Cu at (83.9, 96.7)
- added C18: 10n, Capacitor_SMD:C_0805_2012Metric_Pad1.18x1.45mm_HandSolder, B.Cu at (84.7, 98.0)
- added C19: 10n, Capacitor_SMD:C_0805_2012Metric_Pad1.18x1.45mm_HandSolder, F.Cu at (91.0, 93.9)
- added C20: 100n, Capacitor_SMD:C_0805_2012Metric_Pad1.18x1.45mm_HandSolder, F.Cu at (81.3, 91.5)
- added C21: 36p, Capacitor_SMD:C_0805_2012Metric_Pad1.18x1.45mm_HandSolder, F.Cu at (94.0, 98.4)
- added C22: 36p, Capacitor_SMD:C_0805_2012Metric_Pad1.18x1.45mm_HandSolder, F.Cu at (97.0, 99.6)
- added C23: 100n, Capacitor_SMD:C_0805_2012Metric_Pad1.18x1.45mm_HandSolder, F.Cu at (78.1, 88.6)
- added C24: 68p, Capacitor_SMD:C_0805_2012Metric_Pad1.18x1.45mm_HandSolder, F.Cu at (80.5, 109.6)
- added C25: 15p, Capacitor_SMD:C_0805_2012Metric_Pad1.18x1.45mm_HandSolder, F.Cu at (82.2, 109.7)
- added C26: 470p, Capacitor_SMD:C_0805_2012Metric_Pad1.18x1.45mm_HandSolder, F.Cu at (78.6, 109.6)
- added C27: 18p, Capacitor_SMD:C_0805_2012Metric_Pad1.18x1.45mm_HandSolder, F.Cu at (77.8, 106.7)
- added C28: 18p, Capacitor_SMD:C_0805_2012Metric_Pad1.18x1.45mm_HandSolder, F.Cu at (77.7, 112.6)
- added C29: 180p, Capacitor_SMD:C_0805_2012Metric_Pad1.18x1.45mm_HandSolder, F.Cu at (69.0, 106.1)
- added C30: 180p, Capacitor_SMD:C_0805_2012Metric_Pad1.18x1.45mm_HandSolder, F.Cu at (68.9, 114.0)
- added C31: 9p, Capacitor_SMD:C_0805_2012Metric_Pad1.18x1.45mm_HandSolder, F.Cu at (51.4, 125.3)
- added C32: 10n, Capacitor_SMD:C_0805_2012Metric_Pad1.18x1.45mm_HandSolder, F.Cu at (96.0, 118.0)
- added C34: 100n, Capacitor_SMD:C_0805_2012Metric_Pad1.18x1.45mm_HandSolder, F.Cu at (77.9, 80.4)
- added C36: 10n, Capacitor_SMD:C_0805_2012Metric_Pad1.18x1.45mm_HandSolder, F.Cu at (60.1, 126.2)
- added C37: 100n, Capacitor_SMD:C_0805_2012Metric_Pad1.18x1.45mm_HandSolder, F.Cu at (56.9, 123.2)
- added C38: 100n, Capacitor_SMD:C_0805_2012Metric_Pad1.18x1.45mm_HandSolder, F.Cu at (61.1, 123.2)
- added C39: 33p, Capacitor_SMD:C_0805_2012Metric_Pad1.18x1.45mm_HandSolder, F.Cu at (69.0, 108.1)
- added C40: 33p, Capacitor_SMD:C_0805_2012Metric_Pad1.18x1.45mm_HandSolder, F.Cu at (68.9, 116.1)
- added C9: 10n, Capacitor_SMD:C_0805_2012Metric_Pad1.18x1.45mm_HandSolder, F.Cu at (49.9, 128.3)
- added R1: 5k, Resistor_SMD:R_0805_2012Metric_Pad1.20x1.40mm_HandSolder, F.Cu at (67.6, 93.1)
- added R10: 1.2k, Resistor_SMD:R_0805_2012Metric_Pad1.20x1.40mm_HandSolder, F.Cu at (89.0, 127.7)
- added R11: 470, Resistor_SMD:R_0805_2012Metric_Pad1.20x1.40mm_HandSolder, F.Cu at (80.0, 80.4)
- added R12: BP, Resistor_SMD:R_0805_2012Metric_Pad1.20x1.40mm_HandSolder, F.Cu at (85.7, 122.5)
- added R13: 2k5, Resistor_SMD:R_0805_2012Metric_Pad1.20x1.40mm_HandSolder, F.Cu at (54.7, 117.2)
- added R14: 19k, Resistor_SMD:R_0805_2012Metric_Pad1.20x1.40mm_HandSolder, F.Cu at (49.9, 122.4)
- added R15: 31k, Resistor_SMD:R_0805_2012Metric_Pad1.20x1.40mm_HandSolder, F.Cu at (50.0, 130.3)
- added R16: 27, Resistor_SMD:R_0805_2012Metric_Pad1.20x1.40mm_HandSolder, B.Cu at (62.4, 88.7)
- added R17: 39, Resistor_SMD:R_0805_2012Metric_Pad1.20x1.40mm_HandSolder, B.Cu at (64.3, 88.7)
- added R18: 47, Resistor_SMD:R_0805_2012Metric_Pad1.20x1.40mm_HandSolder, F.Cu at (65.7, 84.6)
- added R19: 33, Resistor_SMD:R_0805_2012Metric_Pad1.20x1.40mm_HandSolder, B.Cu at (60.2, 89.8)
- added R2: 5k, Resistor_SMD:R_0805_2012Metric_Pad1.20x1.40mm_HandSolder, F.Cu at (69.7, 84.6)
- added R20: 10, Resistor_SMD:R_0805_2012Metric_Pad1.20x1.40mm_HandSolder, B.Cu at (66.7, 89.8)
- added R21: 3, Resistor_SMD:R_0805_2012Metric_Pad1.20x1.40mm_HandSolder, F.Cu at (68.5, 86.6)
- added R22: 27, Resistor_SMD:R_0805_2012Metric_Pad1.20x1.40mm_HandSolder, B.Cu at (62.2, 92.1)
- added R23: 39, Resistor_SMD:R_0805_2012Metric_Pad1.20x1.40mm_HandSolder, B.Cu at (64.1, 92.1)
- added R24: 47, Resistor_SMD:R_0805_2012Metric_Pad1.20x1.40mm_HandSolder, F.Cu at (67.6, 89.4)
- added R25: 100, Resistor_SMD:R_0805_2012Metric_Pad1.20x1.40mm_HandSolder, F.Cu at (59.1, 123.2)
- added R26: BP, Resistor_SMD:R_1206_3216Metric_Pad1.30x1.75mm_HandSolder, F.Cu at (61.4, 83.7)
- added R27: BP, Resistor_SMD:R_1206_3216Metric_Pad1.30x1.75mm_HandSolder, F.Cu at (53.5, 92.2)
- added R28: BP, Resistor_SMD:R_1206_3216Metric_Pad1.30x1.75mm_HandSolder, F.Cu at (70.3, 101.8)
- added R29: BP, Resistor_SMD:R_1206_3216Metric_Pad1.30x1.75mm_HandSolder, F.Cu at (56.3, 99.9)
- added R3: 10k, Resistor_SMD:R_0805_2012Metric_Pad1.20x1.40mm_HandSolder, F.Cu at (68.2, 126.7)
- added R30: BP, Resistor_SMD:R_1206_3216Metric_Pad1.30x1.75mm_HandSolder, F.Cu at (88.1, 106.5)
- added R31: BP, Resistor_SMD:R_1206_3216Metric_Pad1.30x1.75mm_HandSolder, F.Cu at (90.6, 106.5)
- added R32: BP, Resistor_SMD:R_1206_3216Metric_Pad1.30x1.75mm_HandSolder, F.Cu at (57.2, 108.1)
- added R33: BP, Resistor_SMD:R_1206_3216Metric_Pad1.30x1.75mm_HandSolder, F.Cu at (57.2, 110.5)
- added R34: BP, Resistor_SMD:R_1206_3216Metric_Pad1.30x1.75mm_HandSolder, F.Cu at (57.2, 112.9)
- added R35: BP, Resistor_SMD:R_1206_3216Metric_Pad1.30x1.75mm_HandSolder, F.Cu at (85.3, 125.1)
- added R36: BP, Resistor_SMD:R_1206_3216Metric_Pad1.30x1.75mm_HandSolder, F.Cu at (45.0, 124.0)
- added R37: BP, Resistor_SMD:R_1206_3216Metric_Pad1.30x1.75mm_HandSolder, F.Cu at (45.0, 126.3)
- added R38: BP, Resistor_SMD:R_1206_3216Metric_Pad1.30x1.75mm_HandSolder, F.Cu at (58.4, 130.9)
- added R39: BP, Resistor_SMD:R_1206_3216Metric_Pad1.30x1.75mm_HandSolder, F.Cu at (58.4, 128.5)
- added R4: 100, Resistor_SMD:R_0805_2012Metric_Pad1.20x1.40mm_HandSolder, F.Cu at (72.3, 86.6)
- added R40: BP, Resistor_SMD:R_1206_3216Metric_Pad1.30x1.75mm_HandSolder, F.Cu at (94.9, 128.3)
- added R41: BP, Resistor_SMD:R_1206_3216Metric_Pad1.30x1.75mm_HandSolder, F.Cu at (84.0, 127.7)
- added R42: 19k, Resistor_SMD:R_0805_2012Metric_Pad1.20x1.40mm_HandSolder, F.Cu at (97.9, 124.3)
- added R43: 19k, Resistor_SMD:R_0805_2012Metric_Pad1.20x1.40mm_HandSolder, F.Cu at (91.7, 131.1)
- added R5: 28k, Resistor_SMD:R_0805_2012Metric_Pad1.20x1.40mm_HandSolder, F.Cu at (74.4, 92.5)
- added R6: 31k, Resistor_SMD:R_0805_2012Metric_Pad1.20x1.40mm_HandSolder, F.Cu at (74.4, 94.4)
- added R7: 5k, Resistor_SMD:R_0805_2012Metric_Pad1.20x1.40mm_HandSolder, F.Cu at (72.8, 104.0)
- added R8: 100, Resistor_SMD:R_0805_2012Metric_Pad1.20x1.40mm_HandSolder, F.Cu at (79.2, 91.5)
- added R9: 1.2k, Resistor_SMD:R_0805_2012Metric_Pad1.20x1.40mm_HandSolder, F.Cu at (90.9, 121.6)
- Y1: moved to B.Cu
- moved C1 120.8 mm to (44.5, 87.2)
- moved C4 120.8 mm to (58.1, 87.2)
- moved J1 120.8 mm to (39.4, 83.5)
- moved L1 120.8 mm to (46.0, 83.9)
- moved L3 120.8 mm to (56.4, 83.9)
- moved C2 120.8 mm to (47.7, 87.2)
- moved C3 120.8 mm to (52.9, 87.2)
- moved L2 120.8 mm to (51.2, 83.9)
- moved D1 98.3 mm to (82.0, 80.4), turned to 90 degrees
- moved TP1 93.4 mm to (56.9, 80.8)
- moved H4 91.1 mm to (100.0, 77.0)
- moved TP2 90.8 mm to (61.4, 80.6)
- moved U4 90.8 mm to (63.8, 89.5), turned to 270 degrees
- moved L11 88.1 mm to (81.4, 106.7), turned to 180 degrees
- moved L13 85.4 mm to (73.4, 107.3), turned to 180 degrees
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Connections:
- D1 pad 2: (no net) -> Net-(D1-Pad2)
- L10 pad 2: (no net) -> Net-(L10-Pad2)
- L11 pad 2: (no net) -> Net-(C26-Pad1)
- L12 pad 2: (no net) -> Net-(C26-Pad2)
- L13 pad 1: (no net) -> Net-(C27-Pad1)
- L14 pad 1: (no net) -> Net-(C28-Pad1)
- L9 pad 1: (no net) -> Net-(C13-Pad1)
- Q1 pad 1: (no net) -> Net-(C10-Pad1)
- Q2 pad 1: (no net) -> Net-(Q2-Pad1)
- Q2 pad 4: (no net) -> Net-(Q2-Pad4)
- TP12 pad 1: (no net) -> /Sheet5FE3342E/In+
- TP12 pad 2: (no net) -> /Sheet5FE3342E/In-
- TP5 pad 1: (no net) -> /37.4 MHz Amp, and 2nd mixer/IN
- U2 pad 1: (no net) -> Net-(C17-Pad1)
- U2 pad 2: (no net) -> Net-(C18-Pad1)
- U2 pad 6: (no net) -> Net-(C21-Pad2)
- U2 pad 8: (no net) -> Net-(C19-Pad1)
- U3 pad 1: (no net) -> Net-(R10-Pad2)
- U3 pad 2: (no net) -> /Sheet5FE3342E/DC_CM
- U3 pad 4: (no net) -> Net-(R40-Pad2)
- U3 pad 5: (no net) -> Net-(R10-Pad1)
- U3 pad 6: (no net) -> GND
- U3 pad 8: (no net) -> Net-(R12-Pad1)
- U4 pad 11: (no net) -> /Attenuator/10dB_out
- U4 pad 12: (no net) -> /Attenuator/20dB_out
- U4 pad 13: (no net) -> /Attenuator/30dB_out
- U4 pad 3: (no net) -> /Attenuator/30dB_in
- U4 pad 4: (no net) -> /Attenuator/20dB_in
- U4 pad 5: (no net) -> /Attenuator/10dB_in
Routing:
- net +5VA: track 0.00 -> 93.4 mm
- net GNDA: track 23.9 -> 44.5 mm, vias 0 -> 28
- net Net-(C31-Pad1): track 0.00 -> 16.6 mm, vias 0 -> 2
- net Net-(C13-Pad1): track 0.00 -> 15.7 mm, vias 0 -> 2
- net Net-(C19-Pad1): track 0.00 -> 15.7 mm
- net /Sheet5FE333A0/Out-: track 0.00 -> 13.9 mm
- net /Sheet5FE333A0/In-: track 0.00 -> 13.5 mm
- net /Sheet5FE333A0/Out+: track 0.00 -> 13.5 mm
- net Net-(C36-Pad1): track 0.00 -> 13.4 mm, vias 0 -> 2
- net /37.4 MHz BPF/OUT: track 0.00 -> 12.2 mm
- net /37.4 MHz BPF/IN: track 0.00 -> 11.5 mm
- net Net-(J2-Pad1): track 0.00 -> 10.1 mm
- net /Sheet5FE333A0/In+: track 0.00 -> 9.63 mm
- net Net-(C31-Pad2): track 0.00 -> 9.16 mm
- net /Attenuator/ATT_SEL1: track 0.00 -> 8.99 mm
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- added copper zone on B.Cu, net GNDA
Other:
- board outline added: 70 x 65 mm
