File: fpga_int_aux_psu.sch (KiCad schematic (older format))
At the start: 18 parts

Commit message: Progress in programmer sheet
Connections:
- net VCCint renamed +1V8
Changed lines of the file:
@@
 AR Path="/6004B3B4/603D6ACA" Ref="#PWR?"  Part="1"
 AR Path="/6004B3B4/603AAE8B/603D6ACA" Ref="#PWR?"  Part="1"
+AR Path="/603D6ACA" Ref="#PWR?"  Part="1"
 F 0 "#PWR?" H 5000 2450 50  0001 C CNN
 F 1 "GNDD" H 5004 2545 50  0000 C CNN
@@
 	6550 2300 6100 2300
 Wire Wire Line
-	7050 2300 6550 2300
+	7050 2300 6950 2300
 Wire Notes Line
 	6850 2950 4250 2950
@@
 AR Path="/6004B3B4/603D6AE6" Ref="#PWR?"  Part="1"
 AR Path="/6004B3B4/603AAE8B/603D6AE6" Ref="#PWR?"  Part="1"
+AR Path="/603D6AE6" Ref="#PWR?"  Part="1"
 F 0 "#PWR?" H 3000 2700 50  0001 C CNN
 F 1 "+3V3" H 3015 3023 50  0000 C CNN
@@
 AR Path="/6004B3B4/603D6AEC" Ref="#PWR?"  Part="1"
 AR Path="/6004B3B4/603AAE8B/603D6AEC" Ref="#PWR?"  Part="1"
+AR Path="/603D6AEC" Ref="#PWR?"  Part="1"
 F 0 "#PWR?" H 3000 3050 50  0001 C CNN
 F 1 "GNDD" H 3004 3145 50  0000 C CNN
@@
 AR Path="/6004B3B4/603D6B02" Ref="#PWR?"  Part="1"
 AR Path="/6004B3B4/603AAE8B/603D6B02" Ref="#PWR?"  Part="1"
+AR Path="/603D6B02" Ref="#PWR?"  Part="1"
 F 0 "#PWR?" H 5000 3650 50  0001 C CNN
 F 1 "GNDD" H 5004 3745 50  0000 C CNN
@@
 	1    0    0    -1
 $EndComp
+$Comp
+L power:+1V8 #PWR?
+U 1 1 60A1E6CE
+P 6950 2100
+F 0 "#PWR?" H 6950 1950 50  0001 C CNN
+F 1 "+1V8" H 6965 2273 50  0000 C CNN
+F 2 "" H 6950 2100 50  0001 C CNN
+F 3 "" H 6950 2100 50  0001 C CNN
+	1    6950 2100
+	1    0    0    -1
+$EndComp
+Wire Wire Line
+	6950 2100 6950 2300
+Connection ~ 6950 2300
+Wire Wire Line
+	6950 2300 6550 2300
 $EndSCHEMATC

Commit message: Power supply ,,typo" fixes
Parts:
- C? (x2): value C -> 100n
Connections:
- net GNDD: now also C?.2, C?.2
Changed lines of the file:
@@
 AR Path="/6004B3B4/603AAE8B/603D6AD8" Ref="C?"  Part="1"
 F 0 "C?" H 6665 2496 50  0000 L CNN
-F 1 "C" H 6665 2405 50  0000 L CNN
+F 1 "100n" H 6665 2405 50  0000 L CNN
 F 2 "" H 6588 2300 50  0001 C CNN
 F 3 "~" H 6550 2450 50  0001 C CNN
@@
 AR Path="/6004B3B4/603AAE8B/603D6AF9" Ref="C?"  Part="1"
 F 0 "C?" H 6665 3696 50  0000 L CNN
-F 1 "C" H 6665 3605 50  0000 L CNN
+F 1 "100n" H 6665 3605 50  0000 L CNN
 F 2 "" H 6588 3500 50  0001 C CNN
 F 3 "~" H 6550 3650 50  0001 C CNN
@@
 Wire Wire Line
 	6950 2300 6550 2300
+$Comp
+L power:GNDD #PWR?
+U 1 1 60B70727
+P 6550 2600
+F 0 "#PWR?" H 6550 2350 50  0001 C CNN
+F 1 "GNDD" H 6554 2445 50  0000 C CNN
+F 2 "" H 6550 2600 50  0001 C CNN
+F 3 "" H 6550 2600 50  0001 C CNN
+	1    6550 2600
+	1    0    0    -1
+$EndComp
+$Comp
+L power:GNDD #PWR?
+U 1 1 60B709EA
+P 6550 3800
+F 0 "#PWR?" H 6550 3550 50  0001 C CNN
+F 1 "GNDD" H 6554 3645 50  0000 C CNN
+F 2 "" H 6550 3800 50  0001 C CNN
+F 3 "" H 6550 3800 50  0001 C CNN
+	1    6550 3800
+	1    0    0    -1
+$EndComp
 $EndSCHEMATC

Commit message: Power suppley fixes
Connections:
- net +3V3 renamed V_IN
Changed lines of the file:
@@
 Filter at SMPS
-$Comp
-L power:+3V3 #PWR?
-U 1 1 603D6AE6
-P 3000 2850
-AR Path="/6004B3B4/603D6AE6" Ref="#PWR?"  Part="1"
-AR Path="/6004B3B4/603AAE8B/603D6AE6" Ref="#PWR?"  Part="1"
-AR Path="/603D6AE6" Ref="#PWR?"  Part="1"
-F 0 "#PWR?" H 3000 2700 50  0001 C CNN
-F 1 "+3V3" H 3015 3023 50  0000 C CNN
-F 2 "" H 3000 2850 50  0001 C CNN
-F 3 "" H 3000 2850 50  0001 C CNN
-	1    3000 2850
-	1    0    0    -1
-$EndComp
 $Comp
 L power:GNDD #PWR?
@@
 EN_VCCaux
 $Comp
-L power:+3.3V #PWR?
-U 1 1 603DCFE1
-P 3750 2600
-F 0 "#PWR?" H 3750 2450 50  0001 C CNN
-F 1 "+3.3V" H 3765 2773 50  0000 C CNN
-F 2 "" H 3750 2600 50  0001 C CNN
-F 3 "" H 3750 2600 50  0001 C CNN
-	1    3750 2600
-	1    0    0    -1
-$EndComp
-$Comp
 L power:+1V8 #PWR?
 U 1 1 60A1E6CE
@@
 	1    0    0    -1
 $EndComp
+Text HLabel 2750 2600 0    50   Input ~ 0
+V_IN
+Wire Wire Line
+	3750 2600 2750 2600
+Wire Wire Line
+	2750 2600 2750 2850
+Wire Wire Line
+	2750 2850 3000 2850
 $EndSCHEMATC
