File: sdr.sch (KiCad schematic (older format))
At the start: 26 parts

Commit message: Power suppley fixes
Parts:
- added FB?: Ferrite_Bead, symbol Device:Ferrite_Bead
Connections:
- net +3.3VA: now also FB?.1
- net +3V3: now also FB?.2
Other:
- moved on the sheet: C?, K?A, R?, U?
